File: kicad/powersupply/OSDEHA_PSU/OSDEHA_PSU.kicad_sch (KiCad schematic)
At the start: 0 parts

Commit message: up
Parts:
- added J1: PSU HV, Connector_Molex:Molex_KK-396_5273-04A_1x04_P3.96mm_Vertical, symbol Connector:Conn_01x04_Socket
- added T1: Transformer_1P_2S, symbol Device:Transformer_1P_2S
Connections:
- new net GND: J1.4 (Pin_4)
- new net HV_STABI1/AC1: T1.3 (SA)
- new net HV_STABI1/AC2: T1.4 (SB)
- new net HV_STABI1/DC+: J1.1 (Pin_1)
- new net HV_STABI2/AC1: T1.5 (SC)
- new net HV_STABI2/AC2: T1.6 (SD)
- new net HV_STABI2/DC-: J1.2 (Pin_2)
Other:
- removed sheet HV_PSU
- added sheet HV_STABI1 (hv_stabi.kicad_sch)
- added sheet HV_STABI2 (hv_stabi.kicad_sch)
- note added: "GLB"
- note added: "GRID BIAS"
- note added: "PE+CHASSIS"
