File: kicad/amplifier/buffer_CCS_load.kicad_sch (KiCad schematic)
At the start: 3 parts, among them Q9 DN2540

Commit message: UP
Parts:
- renumbered R29 to R31, R30 to R32
Changed lines of the file:
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@@
   (symbol (lib_id "Device:R") (at 137.16 93.98 180) (unit 1)
     (in_bom yes) (on_board yes) (dnp no)
-    (property "Reference" "R30" (at 134.62 93.98 90)
+    (property "Reference" "R32" (at 134.62 93.98 90)
       (effects (font (size 1.27 1.27)))
     )
@@
       (project "OSDEHA_AMP"
         (path "/59cc4414-299b-49db-9f9a-b06f69a12073/964c5f27-279d-4094-beed-423757c37563"
-          (reference "R30") (unit 1)
+          (reference "R32") (unit 1)
         )
         (path "/59cc4414-299b-49db-9f9a-b06f69a12073/117f0db4-f368-407f-8708-b67954482099"
-          (reference "R32") (unit 1)
+          (reference "R34") (unit 1)
         )
       )
@@
   (symbol (lib_id "Device:R") (at 129.54 88.9 180) (unit 1)
     (in_bom yes) (on_board yes) (dnp no)
-    (property "Reference" "R29" (at 127 88.9 90)
+    (property "Reference" "R31" (at 127 88.9 90)
       (effects (font (size 1.27 1.27)))
     )
@@
       (project "OSDEHA_AMP"
         (path "/59cc4414-299b-49db-9f9a-b06f69a12073/964c5f27-279d-4094-beed-423757c37563"
-          (reference "R29") (unit 1)
+          (reference "R31") (unit 1)
         )
         (path "/59cc4414-299b-49db-9f9a-b06f69a12073/117f0db4-f368-407f-8708-b67954482099"
-          (reference "R31") (unit 1)
+          (reference "R33") (unit 1)
         )
       )

Commit message: up
Parts:
- Q9: MPN (none) -> DN2540N5-G
Changed lines of the file:
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@@
       (effects (font (size 1.27 1.27)) hide)
     )
-    (property "Datasheet" "https://www.mouser.ch/ProductDetail/Microchip-Technology/DN2540N5-G?qs=F9TAcTrDwItjOowozNtDSg%3D%3D" (at 134.62 97.79 0)
+    (property "Datasheet" "" (at 134.62 97.79 0)
       (effects (font (size 1.27 1.27)) hide)
     )
-    (property "Sim.Device" "" (at 134.62 102.235 0)
+    (property "MPN" "DN2540N5-G" (at 134.62 85.09 0)
       (effects (font (size 1.27 1.27)) hide)
     )
-    (property "Sim.Type" "VDMOS" (at 134.62 104.14 0)
-      (effects (font (size 1.27 1.27)) hide)
-    )
-    (property "Sim.Pins" "1=D 2=G 3=S" (at 134.62 100.33 0)
-      (effects (font (size 1.27 1.27)) hide)
-    )

Commit message: up
Parts:
- removed R31: 100, Resistor_THT:R_Axial_DIN0207_L6.3mm_D2.5mm_P10.16mm_Horizontal, symbol Device:R
- added D11, D12: 15V, Diode_THT:D_DO-41_SOD81_P7.62mm_Horizontal, symbol Device:D_Zener
- added R21: 300, Resistor_THT:R_Axial_DIN0207_L6.3mm_D2.5mm_P10.16mm_Horizontal, symbol Device:R
Connections:
- net NEG: now also R21.1
- net at Q9.3 (S), R32.2: now also D12.1 (K)
- net at Q9.2 (G): now also D11.1 (K), R21.2
- new net: D11.2 (A), D12.2 (A)
Other:
- moved on the sheet: R32
Changed lines of the file:
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@@
 (kicad_sch (version 20230121) (generator eeschema)
   (paper "A4")
-  (junction (at 137.16 97.79) (diameter 0) (color 0 0 0 0)
+  (junction (at 121.92 90.17) (diameter 0) (color 0 0 0 0)
   )
-  (wire (pts (xy 129.54 97.79) (xy 137.16 97.79))
+  (junction (at 137.16 102.87) (diameter 0) (color 0 0 0 0)
+  )
+  (junction (at 137.16 90.17) (diameter 0) (color 0 0 0 0)
+  )
+  (wire (pts (xy 137.16 101.6) (xy 137.16 102.87))
     (stroke (width 0) (type default))
   )
-  (wire (pts (xy 137.16 97.79) (xy 137.16 99.06))
+  (wire (pts (xy 129.54 85.09) (xy 121.92 85.09))
     (stroke (width 0) (type default))
   )
-  (wire (pts (xy 129.54 92.71) (xy 129.54 97.79))
+  (wire (pts (xy 121.92 90.17) (xy 121.92 93.98))
+    (stroke (width 0) (type default))
+  )
+  (wire (pts (xy 121.92 101.6) (xy 121.92 102.87))
+    (stroke (width 0) (type default))
+  )
+  (wire (pts (xy 121.92 102.87) (xy 137.16 102.87))
+    (stroke (width 0) (type default))
+  )
+  (wire (pts (xy 137.16 102.87) (xy 137.16 105.41))
+    (stroke (width 0) (type default))
+  )
+  (wire (pts (xy 137.16 93.98) (xy 137.16 90.17))
+    (stroke (width 0) (type default))
+  )
+  (wire (pts (xy 121.92 85.09) (xy 121.92 90.17))
     (stroke (width 0) (type default))
   )
@@
     (effects (font (size 1.27 1.27)) (justify left bottom))
   )
-  (hierarchical_label "NEG" (shape passive) (at 137.16 99.06 270) (fields_autoplaced)
+  (hierarchical_label "NEG" (shape passive) (at 137.16 105.41 270) (fields_autoplaced)
     (effects (font (size 1.27 1.27)) (justify right))
   )
@@
     (effects (font (size 1.27 1.27)) (justify left))
   )
-  (symbol (lib_id "Device:R") (at 137.16 93.98 180) (unit 1)
+  (symbol (lib_id "Device:R") (at 137.16 97.79 180) (unit 1)
     (in_bom yes) (on_board yes) (dnp no)
-    (property "Reference" "R32" (at 134.62 93.98 90)
+    (property "Reference" "R32" (at 134.62 97.79 90)
       (effects (font (size 1.27 1.27)))
     )
-    (property "Value" "150" (at 137.16 93.98 90)
+    (property "Value" "150" (at 137.16 97.79 90)
       (effects (font (size 1.27 1.27)))
     )
-    (property "Footprint" "Resistor_THT:R_Axial_DIN0207_L6.3mm_D2.5mm_P10.16mm_Horizontal" (at 138.938 93.98 90)
+    (property "Footprint" "Resistor_THT:R_Axial_DIN0207_L6.3mm_D2.5mm_P10.16mm_Horizontal" (at 138.938 97.79 90)
       (effects (font (size 1.27 1.27)) hide)
     )
-    (property "Datasheet" "~" (at 137.16 93.98 0)
+    (property "Datasheet" "~" (at 137.16 97.79 0)
       (effects (font (size 1.27 1.27)) hide)
     )
@@
         (path "/59cc4414-299b-49db-9f9a-b06f69a12073/117f0db4-f368-407f-8708-b67954482099"
           (reference "R34") (unit 1)
+        )
+      )
+    )
+  )
+  (symbol (lib_id "Device:R") (at 121.92 97.79 180) (unit 1)
+    (in_bom yes) (on_board yes) (dnp no)
+    (property "Reference" "R21" (at 120.015 95.885 90)
+      (effects (font (size 1.27 1.27)) (justify left))
+    )
+    (property "Value" "300" (at 121.92 97.79 90)
+      (effects (font (size 1.27 1.27)))
+    )
+    (property "Footprint" "Resistor_THT:R_Axial_DIN0207_L6.3mm_D2.5mm_P10.16mm_Horizontal" (at 123.698 97.79 90)
+      (effects (font (size 1.27 1.27)) hide)
+    )
+    (property "Datasheet" "~" (at 121.92 97.79 0)
+      (effects (font (size 1.27 1.27)) hide)
+    )
+    (pin "1")
+    (pin "2")
+    (instances
+      (project "OSDEHA_AMP"
+        (path "/59cc4414-299b-49db-9f9a-b06f69a12073/964c5f27-279d-4094-beed-423757c37563"
+          (reference "R21") (unit 1)
+        )
+        (path "/59cc4414-299b-49db-9f9a-b06f69a12073/117f0db4-f368-407f-8708-b67954482099"
+          (reference "R31") (unit 1)
         )
       )
@@
     )
   )
-  (symbol (lib_id "Device:R") (at 129.54 88.9 180) (unit 1)
+  (symbol (lib_id "Device:D_Zener") (at 125.73 90.17 0) (unit 1)
     (in_bom yes) (on_board yes) (dnp no)
-    (property "Reference" "R31" (at 127 88.9 90)
+    (property "Reference" "D11" (at 123.19 92.71 0)
       (effects (font (size 1.27 1.27)))
     )
-    (property "Value" "100" (at 129.54 88.9 90)
+    (property "Value" "15V" (at 127 92.71 0)
       (effects (font (size 1.27 1.27)))
     )
-    (property "Footprint" "Resistor_THT:R_Axial_DIN0207_L6.3mm_D2.5mm_P10.16mm_Horizontal" (at 131.318 88.9 90)
+    (property "Footprint" "Diode_THT:D_DO-41_SOD81_P7.62mm_Horizontal" (at 125.73 90.17 0)
       (effects (font (size 1.27 1.27)) hide)
     )
-    (property "Datasheet" "~" (at 129.54 88.9 0)
+    (property "Datasheet" "~" (at 125.73 90.17 0)
       (effects (font (size 1.27 1.27)) hide)
     )
+    (property "MPN" "ZY15" (at 125.73 90.17 0)
+      (effects (font (size 1.27 1.27)) hide)
+    )
+    (pin "2")
     (pin "1")
-    (pin "2")
     (instances
       (project "OSDEHA_AMP"
         (path "/59cc4414-299b-49db-9f9a-b06f69a12073/964c5f27-279d-4094-beed-423757c37563"
-          (reference "R31") (unit 1)
+          (reference "D11") (unit 1)
         )
         (path "/59cc4414-299b-49db-9f9a-b06f69a12073/117f0db4-f368-407f-8708-b67954482099"
-          (reference "R33") (unit 1)
+          (reference "D13") (unit 1)
         )
       )
+    )
+  )
+  (symbol (lib_id "Device:D_Zener") (at 133.35 90.17 0) (mirror y) (unit 1)
+    (in_bom yes) (on_board yes) (dnp no)
+    (property "Reference" "D12" (at 135.89 92.71 0)
+      (effects (font (size 1.27 1.27)))
+    )
+    (property "Value" "15V" (at 132.08 92.71 0)
+      (effects (font (size 1.27 1.27)))
+    )
+    (property "Footprint" "Diode_THT:D_DO-41_SOD81_P7.62mm_Horizontal" (at 133.35 90.17 0)
+      (effects (font (size 1.27 1.27)) hide)
+    )
+    (property "Datasheet" "~" (at 133.35 90.17 0)
+      (effects (font (size 1.27 1.27)) hide)
+    )
+    (property "MPN" "ZY15" (at 133.35 90.17 0)
+      (effects (font (size 1.27 1.27)) hide)
+    )
+    (pin "2")
+    (pin "1")
+    (instances
+      (project "OSDEHA_AMP"
+        (path "/59cc4414-299b-49db-9f9a-b06f69a12073/964c5f27-279d-4094-beed-423757c37563"
+          (reference "D12") (unit 1)
+        )
+        (path "/59cc4414-299b-49db-9f9a-b06f69a12073/117f0db4-f368-407f-8708-b67954482099"
+          (reference "D14") (unit 1)
+        )
+      )

Commit message: up
Parts:
- renumbered R21 to R33, R32 to R34
Changed lines of the file:
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@@
   (symbol (lib_id "Device:R") (at 137.16 97.79 180) (unit 1)
     (in_bom yes) (on_board yes) (dnp no)
-    (property "Reference" "R32" (at 134.62 97.79 90)
+    (property "Reference" "R34" (at 134.62 97.79 90)
       (effects (font (size 1.27 1.27)))
     )
@@
       (project "OSDEHA_AMP"
         (path "/59cc4414-299b-49db-9f9a-b06f69a12073/964c5f27-279d-4094-beed-423757c37563"
-          (reference "R32") (unit 1)
+          (reference "R34") (unit 1)
         )
         (path "/59cc4414-299b-49db-9f9a-b06f69a12073/117f0db4-f368-407f-8708-b67954482099"
-          (reference "R34") (unit 1)
+          (reference "R36") (unit 1)
         )
       )
@@
   (symbol (lib_id "Device:R") (at 121.92 97.79 180) (unit 1)
     (in_bom yes) (on_board yes) (dnp no)
-    (property "Reference" "R21" (at 120.015 95.885 90)
+    (property "Reference" "R33" (at 120.015 95.885 90)
       (effects (font (size 1.27 1.27)) (justify left))
     )
@@
       (project "OSDEHA_AMP"
         (path "/59cc4414-299b-49db-9f9a-b06f69a12073/964c5f27-279d-4094-beed-423757c37563"
-          (reference "R21") (unit 1)
+          (reference "R33") (unit 1)
         )
         (path "/59cc4414-299b-49db-9f9a-b06f69a12073/117f0db4-f368-407f-8708-b67954482099"
-          (reference "R31") (unit 1)
+          (reference "R35") (unit 1)
         )
       )

Commit message: up
Parts:
- renumbered R33 to R35, R34 to R36
Changed lines of the file:
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@@
     (stroke (width 0) (type default))
   )
-  (text "10 mA CCS" (at 143.51 95.25 0)
+  (text "10 mA CCS" (at 128.27 71.12 0)
     (effects (font (size 1.27 1.27)) (justify left bottom))
   )
@@
   (symbol (lib_id "Device:R") (at 137.16 97.79 180) (unit 1)
     (in_bom yes) (on_board yes) (dnp no)
-    (property "Reference" "R34" (at 134.62 97.79 90)
+    (property "Reference" "R36" (at 134.62 97.79 90)
       (effects (font (size 1.27 1.27)))
     )
@@
       (project "OSDEHA_AMP"
         (path "/59cc4414-299b-49db-9f9a-b06f69a12073/964c5f27-279d-4094-beed-423757c37563"
-          (reference "R34") (unit 1)
+          (reference "R36") (unit 1)
         )
         (path "/59cc4414-299b-49db-9f9a-b06f69a12073/117f0db4-f368-407f-8708-b67954482099"
-          (reference "R36") (unit 1)
+          (reference "R38") (unit 1)
         )
       )
@@
   (symbol (lib_id "Device:R") (at 121.92 97.79 180) (unit 1)
     (in_bom yes) (on_board yes) (dnp no)
-    (property "Reference" "R33" (at 120.015 95.885 90)
-      (effects (font (size 1.27 1.27)) (justify left))
+    (property "Reference" "R35" (at 119.38 97.79 90)
+      (effects (font (size 1.27 1.27)))
     )
     (property "Value" "300" (at 121.92 97.79 90)
@@
       (project "OSDEHA_AMP"
         (path "/59cc4414-299b-49db-9f9a-b06f69a12073/964c5f27-279d-4094-beed-423757c37563"
-          (reference "R33") (unit 1)
+          (reference "R35") (unit 1)
         )
         (path "/59cc4414-299b-49db-9f9a-b06f69a12073/117f0db4-f368-407f-8708-b67954482099"
-          (reference "R35") (unit 1)
+          (reference "R37") (unit 1)
         )
       )
@@
   (symbol (lib_id "Device:D_Zener") (at 125.73 90.17 0) (unit 1)
     (in_bom yes) (on_board yes) (dnp no)
-    (property "Reference" "D11" (at 123.19 92.71 0)
+    (property "Reference" "D11" (at 125.73 92.71 0)
       (effects (font (size 1.27 1.27)))
     )
-    (property "Value" "15V" (at 127 92.71 0)
+    (property "Value" "15V" (at 125.73 87.63 0)
       (effects (font (size 1.27 1.27)))
     )
@@
   (symbol (lib_id "Device:D_Zener") (at 133.35 90.17 0) (mirror y) (unit 1)
     (in_bom yes) (on_board yes) (dnp no)
-    (property "Reference" "D12" (at 135.89 92.71 0)
+    (property "Reference" "D12" (at 133.35 92.71 0)
       (effects (font (size 1.27 1.27)))
     )
-    (property "Value" "15V" (at 132.08 92.71 0)
+    (property "Value" "15V" (at 132.08 87.63 0)
       (effects (font (size 1.27 1.27)))
     )

Commit message: up
Parts:
- renumbered R35 to R37, R36 to R38
Changed lines of the file:
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@@
   (symbol (lib_id "Device:R") (at 137.16 97.79 180) (unit 1)
     (in_bom yes) (on_board yes) (dnp no)
-    (property "Reference" "R36" (at 134.62 97.79 90)
+    (property "Reference" "R38" (at 134.62 97.79 90)
       (effects (font (size 1.27 1.27)))
     )
@@
       (project "OSDEHA_AMP"
         (path "/59cc4414-299b-49db-9f9a-b06f69a12073/964c5f27-279d-4094-beed-423757c37563"
-          (reference "R36") (unit 1)
+          (reference "R38") (unit 1)
         )
         (path "/59cc4414-299b-49db-9f9a-b06f69a12073/117f0db4-f368-407f-8708-b67954482099"
-          (reference "R38") (unit 1)
+          (reference "R40") (unit 1)
         )
       )
@@
   (symbol (lib_id "Device:R") (at 121.92 97.79 180) (unit 1)
     (in_bom yes) (on_board yes) (dnp no)
-    (property "Reference" "R35" (at 119.38 97.79 90)
+    (property "Reference" "R37" (at 119.38 97.79 90)
       (effects (font (size 1.27 1.27)))
     )
@@
       (project "OSDEHA_AMP"
         (path "/59cc4414-299b-49db-9f9a-b06f69a12073/964c5f27-279d-4094-beed-423757c37563"
-          (reference "R35") (unit 1)
+          (reference "R37") (unit 1)
         )
         (path "/59cc4414-299b-49db-9f9a-b06f69a12073/117f0db4-f368-407f-8708-b67954482099"
-          (reference "R37") (unit 1)
+          (reference "R39") (unit 1)
         )
       )

Commit message: amp pcb
Parts:
- renumbered R37 to R40, R38 to R41
Changed lines of the file:
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@@
   (symbol (lib_id "Device:R") (at 137.16 97.79 180) (unit 1)
     (in_bom yes) (on_board yes) (dnp no)
-    (property "Reference" "R38" (at 134.62 97.79 90)
+    (property "Reference" "R41" (at 134.62 97.79 90)
       (effects (font (size 1.27 1.27)))
     )
@@
       (project "OSDEHA_AMP"
         (path "/59cc4414-299b-49db-9f9a-b06f69a12073/964c5f27-279d-4094-beed-423757c37563"
-          (reference "R38") (unit 1)
+          (reference "R41") (unit 1)
         )
         (path "/59cc4414-299b-49db-9f9a-b06f69a12073/117f0db4-f368-407f-8708-b67954482099"
-          (reference "R40") (unit 1)
+          (reference "R43") (unit 1)
         )
       )
@@
   (symbol (lib_id "Device:R") (at 121.92 97.79 180) (unit 1)
     (in_bom yes) (on_board yes) (dnp no)
-    (property "Reference" "R37" (at 119.38 97.79 90)
+    (property "Reference" "R40" (at 119.38 97.79 90)
       (effects (font (size 1.27 1.27)))
     )
@@
       (project "OSDEHA_AMP"
         (path "/59cc4414-299b-49db-9f9a-b06f69a12073/964c5f27-279d-4094-beed-423757c37563"
-          (reference "R37") (unit 1)
+          (reference "R40") (unit 1)
         )
         (path "/59cc4414-299b-49db-9f9a-b06f69a12073/117f0db4-f368-407f-8708-b67954482099"
-          (reference "R39") (unit 1)
+          (reference "R42") (unit 1)
         )
       )
