File: kicad/amplifier/OSDEHA_AMP.kicad_sch (KiCad schematic)
At the start: 61 parts, among them J1 INPUT, J2 HEATERS DC, J3 PSU HV, J4 OUTPUT, J5 DHT FIL2, J6 DHT FIL1, Q1 DN2540N5-G, Q2 DN2540N5-G, Q3 STF3LN80K5, Q4 STF3LN80K5, SW1 SW_DPDT_x2, U1 6E5P, U2 6E5P, U3 801A, U4 801A

Commit message: amp pcb
Parts:
- renumbered C3 to C1, C4 to C2, C5 to C3, C6 to C4, C1 to C5, C2 to C6, C9 to C7, R41 to R25, R42 to R26, R25 to R27, R26 to R28, R43 to R29
Changed lines of the file:
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@@
   (symbol (lib_id "Device:R") (at 361.95 78.74 0) (unit 1)
     (in_bom yes) (on_board yes) (dnp no)
-    (property "Reference" "R43" (at 364.49 78.74 90)
+    (property "Reference" "R29" (at 364.49 78.74 90)
       (effects (font (size 1.27 1.27)))
     )
@@
       (project "OSDEHA_AMP"
         (path "/59cc4414-299b-49db-9f9a-b06f69a12073"
-          (reference "R43") (unit 1)
+          (reference "R29") (unit 1)
         )
       )
@@
   (symbol (lib_id "Device:C_Polarized") (at 356.87 78.74 0) (unit 1)
     (in_bom yes) (on_board yes) (dnp no)
-    (property "Reference" "C9" (at 356.87 81.28 0)
+    (property "Reference" "C7" (at 356.87 81.28 0)
       (effects (font (size 1.27 1.27)) (justify right))
     )
@@
       (project "OSDEHA_AMP"
         (path "/59cc4414-299b-49db-9f9a-b06f69a12073"
-          (reference "C9") (unit 1)
+          (reference "C7") (unit 1)
         )
       )
@@
   (symbol (lib_id "Device:R") (at 342.9 78.74 0) (unit 1)
     (in_bom yes) (on_board yes) (dnp no)
-    (property "Reference" "R42" (at 345.44 78.74 90)
+    (property "Reference" "R26" (at 345.44 78.74 90)
       (effects (font (size 1.27 1.27)))
     )
@@
       (project "OSDEHA_AMP"
         (path "/59cc4414-299b-49db-9f9a-b06f69a12073"
-          (reference "R42") (unit 1)
+          (reference "R26") (unit 1)
         )
       )
@@
   (symbol (lib_id "Device:C") (at 171.45 166.37 0) (unit 1)
     (in_bom yes) (on_board yes) (dnp no)
-    (property "Reference" "C3" (at 170.18 163.83 0)
+    (property "Reference" "C1" (at 170.18 163.83 0)
       (effects (font (size 1.27 1.27)) (justify right))
     )
@@
       (project "OSDEHA_AMP"
         (path "/59cc4414-299b-49db-9f9a-b06f69a12073"
-          (reference "C3") (unit 1)
+          (reference "C1") (unit 1)
         )
       )
@@
   (symbol (lib_id "Device:R") (at 358.14 121.92 90) (unit 1)
     (in_bom yes) (on_board yes) (dnp no)
-    (property "Reference" "R25" (at 355.6 119.38 90)
+    (property "Reference" "R27" (at 355.6 119.38 90)
       (effects (font (size 1.27 1.27)))
     )
@@
       (project "OSDEHA_AMP"
         (path "/59cc4414-299b-49db-9f9a-b06f69a12073"
-          (reference "R25") (unit 1)
+          (reference "R27") (unit 1)
         )
       )
@@
   (symbol (lib_id "Device:C_Polarized") (at 337.82 78.74 0) (unit 1)
     (in_bom yes) (on_board yes) (dnp no)
-    (property "Reference" "C2" (at 337.82 81.28 0)
+    (property "Reference" "C6" (at 337.82 81.28 0)
       (effects (font (size 1.27 1.27)) (justify right))
     )
@@
       (project "OSDEHA_AMP"
         (path "/59cc4414-299b-49db-9f9a-b06f69a12073"
-          (reference "C2") (unit 1)
+          (reference "C6") (unit 1)
         )
       )
@@
   (symbol (lib_id "Device:C") (at 175.26 143.51 270) (unit 1)
     (in_bom yes) (on_board yes) (dnp no)
-    (property "Reference" "C5" (at 177.8 144.78 90)
+    (property "Reference" "C3" (at 177.8 144.78 90)
       (effects (font (size 1.27 1.27)))
     )
@@
       (project "OSDEHA_AMP"
         (path "/59cc4414-299b-49db-9f9a-b06f69a12073"
-          (reference "C5") (unit 1)
+          (reference "C3") (unit 1)
         )
       )
@@
   (symbol (lib_id "Device:C_Polarized") (at 318.77 78.74 180) (unit 1)
     (in_bom yes) (on_board yes) (dnp no)
-    (property "Reference" "C1" (at 318.77 81.28 0)
+    (property "Reference" "C5" (at 318.77 81.28 0)
       (effects (font (size 1.27 1.27)) (justify left))
     )
@@
       (project "OSDEHA_AMP"
         (path "/59cc4414-299b-49db-9f9a-b06f69a12073"
-          (reference "C1") (unit 1)
+          (reference "C5") (unit 1)
         )
       )
@@
   (symbol (lib_id "Device:C") (at 198.12 166.37 0) (unit 1)
     (in_bom yes) (on_board yes) (dnp no)
-    (property "Reference" "C6" (at 196.85 163.83 0)
+    (property "Reference" "C4" (at 196.85 163.83 0)
       (effects (font (size 1.27 1.27)) (justify right))
     )
@@
       (project "OSDEHA_AMP"
         (path "/59cc4414-299b-49db-9f9a-b06f69a12073"
-          (reference "C6") (unit 1)
+          (reference "C4") (unit 1)
         )
       )
@@
   (symbol (lib_id "Device:R") (at 323.85 78.74 0) (unit 1)
     (in_bom yes) (on_board yes) (dnp no)
-    (property "Reference" "R41" (at 326.39 78.74 90)
+    (property "Reference" "R25" (at 326.39 78.74 90)
       (effects (font (size 1.27 1.27)))
     )
@@
       (project "OSDEHA_AMP"
         (path "/59cc4414-299b-49db-9f9a-b06f69a12073"
-          (reference "R41") (unit 1)
+          (reference "R25") (unit 1)
         )
       )
@@
   (symbol (lib_id "Device:R") (at 358.14 124.46 90) (unit 1)
     (in_bom yes) (on_board yes) (dnp no)
-    (property "Reference" "R26" (at 355.6 127 90)
+    (property "Reference" "R28" (at 355.6 127 90)
       (effects (font (size 1.27 1.27)))
     )
@@
       (project "OSDEHA_AMP"
         (path "/59cc4414-299b-49db-9f9a-b06f69a12073"
-          (reference "R26") (unit 1)
+          (reference "R28") (unit 1)
         )
       )
@@
   (symbol (lib_id "Device:C") (at 175.26 120.65 270) (unit 1)
     (in_bom yes) (on_board yes) (dnp no)
-    (property "Reference" "C4" (at 177.8 121.92 90)
+    (property "Reference" "C2" (at 177.8 121.92 90)
       (effects (font (size 1.27 1.27)))
     )
@@
       (project "OSDEHA_AMP"
         (path "/59cc4414-299b-49db-9f9a-b06f69a12073"
-          (reference "C4") (unit 1)
-        )
-      )
+          (reference "C2") (unit 1)
+        )
+      )

Commit message: MPNs and datasheet links
Parts:
- R1, R3: MPN (none) -> CMF55500K00
- R2, R7: MPN (none) -> CMF551K0000
- R5, R8: MPN (none) -> CMF55300R00
- R6: MPN (none) -> CMF5575R000
Changed lines of the file:
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@@
       (effects (font (size 1.27 1.27)) hide)
     )
-    (property "Datasheet" "~" (at 115.57 173.99 0)
+    (property "Datasheet" "https://www.vishay.com/doc?31018" (at 115.57 173.99 0)
+      (effects (font (size 1.27 1.27)) hide)
+    )
+    (property "MPN" "CMF5575R000" (at 115.57 173.99 90)
       (effects (font (size 1.27 1.27)) hide)
     )
@@
       (effects (font (size 1.27 1.27)) hide)
     )
-    (property "Datasheet" "~" (at 118.11 132.08 0)
+    (property "Datasheet" "https://www.vishay.com/doc?31018" (at 118.11 132.08 0)
+      (effects (font (size 1.27 1.27)) hide)
+    )
+    (property "MPN" "CMF551K0000" (at 118.11 132.08 90)
       (effects (font (size 1.27 1.27)) hide)
     )
@@
       (effects (font (size 1.27 1.27)) hide)
     )
-    (property "Datasheet" "~" (at 85.09 132.08 0)
+    (property "Datasheet" "https://www.vishay.com/doc?31018" (at 85.09 132.08 0)
+      (effects (font (size 1.27 1.27)) hide)
+    )
+    (property "MPN" "CMF551K0000" (at 85.09 132.08 90)
       (effects (font (size 1.27 1.27)) hide)
     )
@@
       (effects (font (size 1.27 1.27)) hide)
     )
-    (property "Datasheet" "~" (at 104.14 167.64 0)
+    (property "Datasheet" "https://diotec.com/request/datasheet/zy1.pdf" (at 104.14 167.64 0)
       (effects (font (size 1.27 1.27)) hide)
     )
@@
       (effects (font (size 1.27 1.27)) hide)
     )
-    (property "Datasheet" "~" (at 100.33 173.99 0)
+    (property "Datasheet" "https://www.vishay.com/doc?31018" (at 100.33 173.99 0)
+      (effects (font (size 1.27 1.27)) hide)
+    )
+    (property "MPN" "CMF55300R00" (at 100.33 173.99 90)
       (effects (font (size 1.27 1.27)) hide)
     )
@@
       (effects (font (size 1.27 1.27)) hide)
     )
-    (property "Datasheet" "~" (at 85.09 149.86 0)
+    (property "Datasheet" "https://www.vishay.com/doc?31018" (at 85.09 149.86 0)
+      (effects (font (size 1.27 1.27)) hide)
+    )
+    (property "MPN" "    CMF55500K00" (at 85.09 149.86 90)
       (effects (font (size 1.27 1.27)) hide)
     )
@@
       (effects (font (size 1.27 1.27)) hide)
     )
-    (property "Datasheet" "~" (at 77.47 149.86 0)
+    (property "Datasheet" "https://www.vishay.com/doc?31018" (at 77.47 149.86 0)
+      (effects (font (size 1.27 1.27)) hide)
+    )
+    (property "MPN" "    CMF55500K00" (at 77.47 149.86 90)
       (effects (font (size 1.27 1.27)) hide)
     )
@@
       (effects (font (size 1.27 1.27)) hide)
     )
-    (property "Datasheet" "~" (at 127 152.4 0)
+    (property "Datasheet" "https://www.vishay.com/doc?31018" (at 127 152.4 0)
+      (effects (font (size 1.27 1.27)) hide)
+    )
+    (property "MPN" "CMF55300R00" (at 127 152.4 90)
       (effects (font (size 1.27 1.27)) hide)
     )
@@
       (effects (font (size 1.27 1.27)) hide)
     )
-    (property "Datasheet" "~" (at 111.76 167.64 0)
-      (effects (font (size 1.27 1.27)) hide)
-    )
+    (property "Datasheet" "https://diotec.com/request/datasheet/zy1.pdf" (at 111.76 167.64 0)
+      (effects (font (size 1.27 1.27)) hide)
+    )

Commit message: MPNs and datasheets
Parts:
- J1: MPN (none) -> 41791-0849
- R11, R13, R16: MPN (none) -> CMF551M0000
- R12, R17: MPN (none) -> CMF5547K000
- R15, R20: MPN (none) -> CMF5525K000
- R18: MPN (none) -> CMF551M000
- R21, R22, R23, R24: MPN (none) -> CMF551K0000
- R27, R28: MPN (none) -> CMF555K1100
Changed lines of the file:
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@@
       (effects (font (size 1.27 1.27)) hide)
     )
-    (property "Datasheet" "~" (at 191.77 173.99 0)
+    (property "Datasheet" "https://www.vishay.com/doc?31018" (at 191.77 173.99 0)
+      (effects (font (size 1.27 1.27)) hide)
+    )
+    (property "MPN" "CMF5525K000" (at 191.77 173.99 90)
       (effects (font (size 1.27 1.27)) hide)
     )
@@
       (effects (font (size 1.27 1.27)) hide)
     )
-    (property "Datasheet" "~" (at 184.15 173.99 0)
+    (property "Datasheet" "https://www.vishay.com/doc?31018" (at 184.15 173.99 0)
+      (effects (font (size 1.27 1.27)) hide)
+    )
+    (property "MPN" "CMF5547K000" (at 184.15 173.99 90)
       (effects (font (size 1.27 1.27)) hide)
     )
@@
       (effects (font (size 1.27 1.27)) hide)
     )
-    (property "Datasheet" "~" (at 220.98 120.65 0)
+    (property "Datasheet" "https://www.vishay.com/doc?31018" (at 220.98 120.65 0)
+      (effects (font (size 1.27 1.27)) hide)
+    )
+    (property "MPN" "CMF551K0000" (at 220.98 120.65 90)
       (effects (font (size 1.27 1.27)) hide)
     )
@@
       (effects (font (size 1.27 1.27)) hide)
     )
-    (property "Datasheet" "~" (at 261.62 148.59 0)
+    (property "Datasheet" "https://www.vishay.com/doc?31018" (at 261.62 148.59 0)
+      (effects (font (size 1.27 1.27)) hide)
+    )
+    (property "MPN" "CMF551K0000" (at 261.62 148.59 90)
       (effects (font (size 1.27 1.27)) hide)
     )
@@
       (effects (font (size 1.27 1.27)) hide)
     )
-    (property "Datasheet" "~" (at 157.48 173.99 0)
+    (property "Datasheet" "https://www.vishay.com/doc?31018" (at 157.48 173.99 0)
+      (effects (font (size 1.27 1.27)) hide)
+    )
+    (property "MPN" "CMF5547K000" (at 157.48 173.99 90)
       (effects (font (size 1.27 1.27)) hide)
     )
@@
       (effects (font (size 1.27 1.27)) hide)
     )
-    (property "Datasheet" "~" (at 177.8 173.99 0)
+    (property "Datasheet" "https://www.vishay.com/doc?31018" (at 177.8 173.99 0)
+      (effects (font (size 1.27 1.27)) hide)
+    )
+    (property "MPN" "CMF551M0000" (at 177.8 173.99 90)
       (effects (font (size 1.27 1.27)) hide)
     )
@@
       (effects (font (size 1.27 1.27)) hide)
     )
-    (property "Datasheet" "~" (at 165.1 173.99 0)
+    (property "Datasheet" "https://www.vishay.com/doc?31018" (at 165.1 173.99 0)
+      (effects (font (size 1.27 1.27)) hide)
+    )
+    (property "MPN" "CMF5525K000" (at 165.1 173.99 90)
       (effects (font (size 1.27 1.27)) hide)
     )
@@
       (effects (font (size 1.27 1.27)) hide)
     )
-    (property "Datasheet" "~" (at 220.98 143.51 0)
+    (property "Datasheet" "https://www.vishay.com/doc?31018" (at 220.98 143.51 0)
+      (effects (font (size 1.27 1.27)) hide)
+    )
+    (property "MPN" "CMF551K0000" (at 220.98 143.51 90)
       (effects (font (size 1.27 1.27)) hide)
     )
@@
       (effects (font (size 1.27 1.27)) hide)
     )
-    (property "Datasheet" "~" (at 151.13 173.99 0)
+    (property "Datasheet" "https://www.vishay.com/doc?31018" (at 151.13 173.99 0)
+      (effects (font (size 1.27 1.27)) hide)
+    )
+    (property "MPN" "CMF551M0000" (at 151.13 173.99 90)
       (effects (font (size 1.27 1.27)) hide)
     )
@@
       (effects (font (size 1.27 1.27)) hide)
     )
-    (property "Datasheet" "~" (at 228.6 125.73 0)
+    (property "Datasheet" "https://diotec.com/request/datasheet/zy1.pdf" (at 228.6 125.73 0)
       (effects (font (size 1.27 1.27)) hide)
     )
@@
       (effects (font (size 1.27 1.27)) hide)
     )
-    (property "Datasheet" "~" (at 161.29 168.91 0)
+    (property "Datasheet" "https://www.mouser.ch/datasheet/2/54/3296-776415.pdf" (at 161.29 168.91 0)
       (effects (font (size 1.27 1.27)) hide)
     )
@@
       (effects (font (size 1.27 1.27)) hide)
     )
-    (property "Datasheet" "~" (at 358.14 121.92 0)
+    (property "Datasheet" "https://www.vishay.com/doc?31018" (at 358.14 121.92 0)
+      (effects (font (size 1.27 1.27)) hide)
+    )
+    (property "MPN" "CMF555K1100" (at 358.14 121.92 90)
       (effects (font (size 1.27 1.27)) hide)
     )
@@
       (effects (font (size 1.27 1.27)) hide)
     )
-    (property "Datasheet" "~" (at 187.96 168.91 0)
+    (property "Datasheet" "https://www.mouser.ch/datasheet/2/54/3296-776415.pdf" (at 187.96 168.91 0)
       (effects (font (size 1.27 1.27)) hide)
     )
@@
       (effects (font (size 1.27 1.27)) hide)
     )
-    (property "Datasheet" "~" (at 308.61 148.59 0)
+    (property "Datasheet" "https://www.vishay.com/doc?31018" (at 308.61 148.59 0)
+      (effects (font (size 1.27 1.27)) hide)
+    )
+    (property "MPN" "CMF551K0000" (at 308.61 148.59 90)
       (effects (font (size 1.27 1.27)) hide)
     )
@@
       (effects (font (size 1.27 1.27)) hide)
     )
-    (property "Datasheet" "~" (at 236.22 148.59 0)
+    (property "Datasheet" "https://diotec.com/request/datasheet/zy1.pdf" (at 236.22 148.59 0)
       (effects (font (size 1.27 1.27)) hide)
     )
@@
       (effects (font (size 1.27 1.27)) hide)
     )
-    (property "Datasheet" "~" (at 161.29 152.4 0)
+    (property "Datasheet" "https://www.vishay.com/doc?31018" (at 161.29 152.4 0)
+      (effects (font (size 1.27 1.27)) hide)
+    )
+    (property "MPN" "CMF551M0000" (at 161.29 152.4 90)
       (effects (font (size 1.27 1.27)) hide)
     )
@@
       (effects (font (size 1.27 1.27)) hide)
     )
-    (property "Datasheet" "~" (at 59.69 137.16 0)
+    (property "Datasheet" "https://www.molex.com/en-us/products/part-detail/417910849?display=pdf" (at 59.69 137.16 0)
+      (effects (font (size 1.27 1.27)) hide)
+    )
+    (property "MPN" "41791-0849" (at 59.69 137.16 0)
       (effects (font (size 1.27 1.27)) hide)
     )
@@
       (effects (font (size 1.27 1.27)) hide)
     )
-    (property "Datasheet" "~" (at 236.22 125.73 0)
+    (property "Datasheet" "https://diotec.com/request/datasheet/zy1.pdf" (at 236.22 125.73 0)
       (effects (font (size 1.27 1.27)) hide)
     )
@@
       (effects (font (size 1.27 1.27)) hide)
     )
-    (property "Datasheet" "~" (at 187.96 152.4 0)
+    (property "Datasheet" "https://www.vishay.com/doc?31018" (at 187.96 152.4 0)
+      (effects (font (size 1.27 1.27)) hide)
+    )
+    (property "MPN" "CMF551M000" (at 187.96 152.4 90)
       (effects (font (size 1.27 1.27)) hide)
     )
@@
       (effects (font (size 1.27 1.27)) hide)
     )
-    (property "Datasheet" "~" (at 358.14 124.46 0)
+    (property "Datasheet" "https://www.vishay.com/doc?31018" (at 358.14 124.46 0)
+      (effects (font (size 1.27 1.27)) hide)
+    )
+    (property "MPN" "CMF555K1100" (at 358.14 124.46 90)
       (effects (font (size 1.27 1.27)) hide)
     )
@@
       (effects (font (size 1.27 1.27)) hide)
     )
-    (property "Datasheet" "~" (at 228.6 148.59 0)
-      (effects (font (size 1.27 1.27)) hide)
-    )
+    (property "Datasheet" "https://diotec.com/request/datasheet/zy1.pdf" (at 228.6 148.59 0)
+      (effects (font (size 1.27 1.27)) hide)
+    )

Commit message: MPNs and datasheets
Parts:
- J2, J4, J5, J6: MPN (none) -> 41791-0849
- J3: MPN (none) -> 41791-0851
Changed lines of the file:
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@@
       (effects (font (size 1.27 1.27)) hide)
     )
-    (property "Datasheet" "https://www.mouser.ch/ProductDetail/Molex/41791-0849?qs=z57USrEQgt3onYoexwRNhA%3D%3D" (at 378.46 166.37 0)
+    (property "Datasheet" "https://www.molex.com/en-us/products/part-detail/417910849?display=pdf" (at 378.46 166.37 0)
+      (effects (font (size 1.27 1.27)) hide)
+    )
+    (property "MPN" "41791-0849" (at 378.46 166.37 0)
       (effects (font (size 1.27 1.27)) hide)
     )
@@
       (effects (font (size 1.27 1.27)) hide)
     )
-    (property "Datasheet" "https://www.mouser.ch/ProductDetail/Molex/41791-0849?qs=z57USrEQgt3onYoexwRNhA%3D%3D" (at 378.46 176.53 0)
+    (property "Datasheet" "https://www.molex.com/en-us/products/part-detail/417910849?display=pdf" (at 378.46 176.53 0)
+      (effects (font (size 1.27 1.27)) hide)
+    )
+    (property "MPN" "41791-0849" (at 378.46 176.53 0)
       (effects (font (size 1.27 1.27)) hide)
     )
@@
       (effects (font (size 1.27 1.27)) hide)
     )
-    (property "Datasheet" "~" (at 375.92 217.17 0)
+    (property "Datasheet" "https://www.molex.com/en-us/products/part-detail/417910849?display=pdf" (at 375.92 217.17 0)
+      (effects (font (size 1.27 1.27)) hide)
+    )
+    (property "MPN" "41791-0849" (at 375.92 217.17 0)
       (effects (font (size 1.27 1.27)) hide)
     )
@@
       (effects (font (size 1.27 1.27)) hide)
     )
-    (property "Datasheet" "https://www.mouser.ch/ProductDetail/Molex/41791-0851?qs=LD9zNoQ5lgUDGtVX5jMt3g%3D%3D" (at 378.46 96.52 0)
+    (property "Datasheet" "https://www.molex.com/en-us/products/part-detail/417910851?display=pdf" (at 378.46 96.52 0)
+      (effects (font (size 1.27 1.27)) hide)
+    )
+    (property "MPN" "41791-0851" (at 378.46 96.52 0)
       (effects (font (size 1.27 1.27)) hide)
     )
@@
       (effects (font (size 1.27 1.27)) hide)
     )
-    (property "Datasheet" "https://www.mouser.ch/ProductDetail/Molex/41791-0849?qs=z57USrEQgt3onYoexwRNhA%3D%3D" (at 378.46 121.92 0)
-      (effects (font (size 1.27 1.27)) hide)
-    )
+    (property "Datasheet" "https://www.molex.com/en-us/products/part-detail/417910849?display=pdf" (at 378.46 121.92 0)
+      (effects (font (size 1.27 1.27)) hide)
+    )
+    (property "MPN" "41791-0849" (at 378.46 121.92 0)
+      (effects (font (size 1.27 1.27)) hide)
+    )

Commit message: up
Parts:
- R4, R9: footprint Resistor_THT:R_Axial_DIN0922_L20.0mm_D9.0mm_P7.62mm_Vertical -> Resistor_THT:R_Axial_Power_L25.0mm_W9.0mm_P27.94mm

Commit message: amp pcb
Parts:
- R10: footprint Resistor_THT:R_Axial_Power_L25.0mm_W9.0mm_P7.62mm_Vertical -> Resistor_THT:R_Axial_Power_L25.0mm_W9.0mm_P30.48mm
- R25, R26, R29: footprint Resistor_THT:R_Axial_DIN0207_L6.3mm_D2.5mm_P10.16mm_Horizontal -> Resistor_THT:R_Axial_DIN0207_L6.3mm_D2.5mm_P2.54mm_Vertical
Changed lines of the file:
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@@
       (effects (font (size 1.27 1.27)))
     )
-    (property "Footprint" "Resistor_THT:R_Axial_DIN0207_L6.3mm_D2.5mm_P10.16mm_Horizontal" (at 360.172 78.74 90)
+    (property "Footprint" "Resistor_THT:R_Axial_DIN0207_L6.3mm_D2.5mm_P2.54mm_Vertical" (at 360.172 78.74 90)
       (effects (font (size 1.27 1.27)) hide)
     )
@@
       (effects (font (size 1.27 1.27)))
     )
-    (property "Footprint" "Resistor_THT:R_Axial_DIN0207_L6.3mm_D2.5mm_P10.16mm_Horizontal" (at 341.122 78.74 90)
+    (property "Footprint" "Resistor_THT:R_Axial_DIN0207_L6.3mm_D2.5mm_P2.54mm_Vertical" (at 341.122 78.74 90)
       (effects (font (size 1.27 1.27)) hide)
     )
@@
       (effects (font (size 1.27 1.27)))
     )
-    (property "Footprint" "Resistor_THT:R_Axial_Power_L25.0mm_W9.0mm_P7.62mm_Vertical" (at 132.08 180.848 90)
+    (property "Footprint" "Resistor_THT:R_Axial_Power_L25.0mm_W9.0mm_P30.48mm" (at 132.08 180.848 90)
       (effects (font (size 1.27 1.27)) hide)
     )
@@
       (effects (font (size 1.27 1.27)))
     )
-    (property "Footprint" "Resistor_THT:R_Axial_DIN0207_L6.3mm_D2.5mm_P10.16mm_Horizontal" (at 322.072 78.74 90)
-      (effects (font (size 1.27 1.27)) hide)
-    )
+    (property "Footprint" "Resistor_THT:R_Axial_DIN0207_L6.3mm_D2.5mm_P2.54mm_Vertical" (at 322.072 78.74 90)
+      (effects (font (size 1.27 1.27)) hide)
+    )

Commit message: up
Parts:
- R4, R9: footprint Resistor_THT:R_Axial_Power_L25.0mm_W9.0mm_P27.94mm -> Resistor_THT:R_Radial_Power_L16.1mm_W9.0mm_P7.37mm
Changed lines of the file:
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@@
       (effects (font (size 1.27 1.27)))
     )
-    (property "Footprint" "Resistor_THT:R_Axial_Power_L25.0mm_W9.0mm_P27.94mm" (at 131.318 95.25 90)
+    (property "Footprint" "Resistor_THT:R_Radial_Power_L16.1mm_W9.0mm_P7.37mm" (at 131.318 95.25 90)
       (effects (font (size 1.27 1.27)) hide)
     )
@@
       (effects (font (size 1.27 1.27)))
     )
-    (property "Footprint" "Resistor_THT:R_Axial_Power_L25.0mm_W9.0mm_P27.94mm" (at 98.298 95.25 90)
-      (effects (font (size 1.27 1.27)) hide)
-    )
+    (property "Footprint" "Resistor_THT:R_Radial_Power_L16.1mm_W9.0mm_P7.37mm" (at 98.298 95.25 90)
+      (effects (font (size 1.27 1.27)) hide)
+    )

Commit message: up
Parts:
- added H5: VENTILATION, MountingHole:MountingHole_5mm, symbol Mechanical:MountingHole
- R10: footprint Resistor_THT:R_Axial_Power_L25.0mm_W9.0mm_P30.48mm -> Resistor_THT:R_Radial_Power_L16.1mm_W9.0mm_P7.37mm
Changed lines of the file:
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@@
       (effects (font (size 1.27 1.27)))
     )
-    (property "Footprint" "Resistor_THT:R_Axial_Power_L25.0mm_W9.0mm_P30.48mm" (at 132.08 180.848 90)
+    (property "Footprint" "Resistor_THT:R_Radial_Power_L16.1mm_W9.0mm_P7.37mm" (at 132.08 180.848 90)
       (effects (font (size 1.27 1.27)) hide)
     )
@@
         )
       )
+    )
+  )
+  (symbol (lib_id "Mechanical:MountingHole") (at 36.83 50.8 0) (unit 1)
+    (in_bom yes) (on_board yes) (dnp no) (fields_autoplaced)
+    (property "Reference" "H5" (at 39.37 49.53 0)
+      (effects (font (size 1.27 1.27)) (justify left))
+    )
+    (property "Value" "VENTILATION" (at 39.37 52.07 0)
+      (effects (font (size 1.27 1.27)) (justify left))
+    )
+    (property "Footprint" "MountingHole:MountingHole_5mm" (at 36.83 50.8 0)
+      (effects (font (size 1.27 1.27)) hide)
+    )
+    (property "Datasheet" "~" (at 36.83 50.8 0)
+      (effects (font (size 1.27 1.27)) hide)
+    )
+    (instances
+      (project "OSDEHA_AMP"
+        (path "/59cc4414-299b-49db-9f9a-b06f69a12073"
+          (reference "H5") (unit 1)
+        )
+      )
