File: kicad/amplifier/OSDEHA_AMP.kicad_sch (KiCad schematic)
At the start: 62 parts, among them J1 INPUT, J2 HEATERS DC, J3 PSU HV, J4 OUTPUT, J5 DHT FIL2, J6 DHT FIL1, Q1 DN2540N5-G, Q2 DN2540N5-G, Q3 STF3LN80K5, Q4 STF3LN80K5, SW1 SW_DPDT_x2, U1 6E5P, U2 6E5P, U3 801A, U4 801A

Commit message: pcb
Parts:
- removed R23, R24: 100, Resistor_THT:R_Axial_DIN0207_L6.3mm_D2.5mm_P10.16mm_Horizontal, symbol Device:R
Connections:
- net Buffer_CCS_load1/POS: now also U3.3 (G)
- net Buffer_CCS_load2/POS: now also U4.3 (G)
- net at U1.1 (F1), U2.1 (F1): now also J2.1 (Pin_1); no longer J2.2 (Pin_2)
- net at U1.6 (F2), U2.6 (F2): now also J2.2 (Pin_2); no longer J2.1 (Pin_1)
Other:
- note added: "100R stopper at socket pin"
- note removed: "solder to socket pin"
Changed lines of the file:
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@@
     (title "OSDEHA Amplifier")
   )
+  (junction (at 127 217.17) (diameter 0) (color 0 0 0 0)
+  )
   (junction (at 187.96 120.65) (diameter 0) (color 0 0 0 0)
   )
@@
   (junction (at 184.15 185.42) (diameter 0) (color 0 0 0 0)
   )
-  (junction (at 132.08 217.17) (diameter 0) (color 0 0 0 0)
-  )
   (junction (at 191.77 179.07) (diameter 0) (color 0 0 0 0)
   )
+  (junction (at 132.08 219.71) (diameter 0) (color 0 0 0 0)
+  )
   (junction (at 224.79 120.65) (diameter 0) (color 0 0 0 0)
   )
@@
   )
   (junction (at 337.82 99.06) (diameter 0) (color 0 0 0 0)
-  )
-  (junction (at 127 219.71) (diameter 0) (color 0 0 0 0)
   )
   (junction (at 345.44 179.07) (diameter 0) (color 0 0 0 0)
@@
   (no_connect (at 93.98 139.7))
   (no_connect (at 127 139.7))
-  (wire (pts (xy 292.1 148.59) (xy 304.8 148.59))
-    (stroke (width 0) (type default))
-  )
   (wire (pts (xy 306.07 119.38) (xy 306.07 121.92))
     (stroke (width 0) (type default))
@@
     (stroke (width 0) (type default))
   )
+  (wire (pts (xy 93.98 217.17) (xy 93.98 212.09))
+    (stroke (width 0) (type default))
+  )
   (wire (pts (xy 113.03 132.08) (xy 113.03 144.78))
     (stroke (width 0) (type default))
@@
     (stroke (width 0) (type default))
   )
+  (wire (pts (xy 127 212.09) (xy 127 217.17))
+    (stroke (width 0) (type default))
+  )
   (wire (pts (xy 198.12 162.56) (xy 198.12 161.29))
     (stroke (width 0) (type default))
@@
     (stroke (width 0) (type default))
   )
+  (wire (pts (xy 132.08 212.09) (xy 132.08 219.71))
+    (stroke (width 0) (type default))
+  )
   (wire (pts (xy 356.87 74.93) (xy 372.11 74.93))
     (stroke (width 0) (type default))
@@
     (stroke (width 0) (type default))
   )
+  (wire (pts (xy 262.89 125.73) (xy 262.89 148.59))
+    (stroke (width 0) (type default))
+  )
   (wire (pts (xy 161.29 130.81) (xy 161.29 148.59))
     (stroke (width 0) (type default))
@@
     (stroke (width 0) (type default))
   )
-  (wire (pts (xy 99.06 212.09) (xy 99.06 217.17))
-    (stroke (width 0) (type default))
-  )
   (wire (pts (xy 161.29 156.21) (xy 161.29 161.29))
     (stroke (width 0) (type default))
@@
     (stroke (width 0) (type default))
   )
+  (wire (pts (xy 248.92 162.56) (xy 248.92 148.59))
+    (stroke (width 0) (type default))
+  )
   (wire (pts (xy 356.87 83.82) (xy 356.87 101.6))
     (stroke (width 0) (type default))
@@
     (stroke (width 0) (type default))
   )
-  (wire (pts (xy 240.03 148.59) (xy 257.81 148.59))
-    (stroke (width 0) (type default))
-  )
   (wire (pts (xy 151.13 161.29) (xy 151.13 170.18))
     (stroke (width 0) (type default))
@@
     (stroke (width 0) (type default))
   )
-  (wire (pts (xy 312.42 148.59) (xy 316.23 148.59))
-    (stroke (width 0) (type default))
-  )
   (wire (pts (xy 308.61 105.41) (xy 308.61 109.22))
     (stroke (width 0) (type default))
@@
     (stroke (width 0) (type default))
   )
-  (wire (pts (xy 93.98 212.09) (xy 93.98 219.71))
-    (stroke (width 0) (type default))
-  )
   (wire (pts (xy 198.12 179.07) (xy 274.32 179.07))
     (stroke (width 0) (type default))
@@
     (stroke (width 0) (type default))
   )
-  (wire (pts (xy 292.1 148.59) (xy 292.1 125.73))
-    (stroke (width 0) (type default))
-  )
   (wire (pts (xy 191.77 168.91) (xy 191.77 170.18))
     (stroke (width 0) (type default))
@@
     (stroke (width 0) (type default))
   )
-  (wire (pts (xy 99.06 217.17) (xy 132.08 217.17))
-    (stroke (width 0) (type default))
-  )
   (wire (pts (xy 69.85 139.7) (xy 69.85 144.78))
     (stroke (width 0) (type default))
@@
     (stroke (width 0) (type default))
   )
-  (wire (pts (xy 127 212.09) (xy 127 219.71))
-    (stroke (width 0) (type default))
-  )
   (wire (pts (xy 96.52 99.06) (xy 96.52 115.57))
     (stroke (width 0) (type default))
@@
     (stroke (width 0) (type default))
   )
-  (wire (pts (xy 240.03 125.73) (xy 292.1 125.73))
+  (wire (pts (xy 99.06 219.71) (xy 132.08 219.71))
     (stroke (width 0) (type default))
   )
@@
     (stroke (width 0) (type default))
   )
+  (wire (pts (xy 262.89 148.59) (xy 269.24 148.59))
+    (stroke (width 0) (type default))
+  )
   (wire (pts (xy 313.69 91.44) (xy 313.69 93.98))
     (stroke (width 0) (type default))
@@
     (stroke (width 0) (type default))
   )
+  (wire (pts (xy 127 217.17) (xy 370.84 217.17))
+    (stroke (width 0) (type default))
+  )
   (wire (pts (xy 224.79 143.51) (xy 232.41 143.51))
     (stroke (width 0) (type default))
   )
+  (wire (pts (xy 262.89 125.73) (xy 240.03 125.73))
+    (stroke (width 0) (type default))
+  )
   (wire (pts (xy 213.36 130.81) (xy 240.03 130.81))
     (stroke (width 0) (type default))
@@
     (stroke (width 0) (type default))
   )
+  (wire (pts (xy 99.06 212.09) (xy 99.06 219.71))
+    (stroke (width 0) (type default))
+  )
   (wire (pts (xy 137.16 128.27) (xy 137.16 119.38))
     (stroke (width 0) (type default))
@@
     (stroke (width 0) (type default))
   )
-  (wire (pts (xy 265.43 148.59) (xy 269.24 148.59))
-    (stroke (width 0) (type default))
-  )
   (wire (pts (xy 256.54 95.25) (xy 240.03 95.25))
     (stroke (width 0) (type default))
@@
     (stroke (width 0) (type default))
   )
-  (wire (pts (xy 93.98 219.71) (xy 127 219.71))
-    (stroke (width 0) (type default))
-  )
   (wire (pts (xy 369.57 101.6) (xy 373.38 101.6))
     (stroke (width 0) (type default))
   )
-  (wire (pts (xy 127 219.71) (xy 370.84 219.71))
+  (wire (pts (xy 297.18 148.59) (xy 297.18 162.56))
     (stroke (width 0) (type default))
   )
@@
     (stroke (width 0) (type default))
   )
+  (wire (pts (xy 316.23 148.59) (xy 297.18 148.59))
+    (stroke (width 0) (type default))
+  )
   (wire (pts (xy 303.53 107.95) (xy 323.85 107.95))
     (stroke (width 0) (type default))
   )
-  (wire (pts (xy 132.08 212.09) (xy 132.08 217.17))
-    (stroke (width 0) (type default))
-  )
   (wire (pts (xy 129.54 111.76) (xy 153.67 111.76))
     (stroke (width 0) (type default))
@@
     (stroke (width 0) (type default))
   )
+  (wire (pts (xy 297.18 162.56) (xy 248.92 162.56))
+    (stroke (width 0) (type default))
+  )
   (wire (pts (xy 372.11 96.52) (xy 372.11 107.95))
     (stroke (width 0) (type default))
   )
+  (wire (pts (xy 132.08 219.71) (xy 370.84 219.71))
+    (stroke (width 0) (type default))
+  )
   (wire (pts (xy 104.14 128.27) (xy 104.14 119.38))
     (stroke (width 0) (type default))
@@
     (stroke (width 0) (type default))
   )
-  (wire (pts (xy 132.08 217.17) (xy 370.84 217.17))
+  (wire (pts (xy 248.92 148.59) (xy 240.03 148.59))
+    (stroke (width 0) (type default))
+  )
+  (wire (pts (xy 93.98 217.17) (xy 127 217.17))
     (stroke (width 0) (type default))
   )
@@
     (effects (font (size 1.27 1.27)) (justify right bottom))
   )
+  (text "100R stopper at\nsocket pin" (at 269.24 154.94 0)
+    (effects (font (size 1.27 1.27)) (justify right bottom))
+  )
   (text "0 V" (at 78.74 138.43 0)
     (effects (font (size 1.27 1.27)) (justify left bottom))
@@
   )
   (text "10 mA" (at 95.25 109.22 90)
-    (effects (font (size 1.27 1.27)) (justify left bottom))
-  )
-  (text "solder to\nsocket pin" (at 257.81 154.94 0)
     (effects (font (size 1.27 1.27)) (justify left bottom))
   )
@@
     (effects (font (size 3 3)) (justify right bottom))
   )
-  (text "solder to\nsocket pin" (at 304.8 154.94 0)
-    (effects (font (size 1.27 1.27)) (justify left bottom))
+  (text "100R stopper at\nsocket pin" (at 314.96 154.94 0)
+    (effects (font (size 1.27 1.27)) (justify right bottom))
   )
   (text "COLD" (at 68.58 142.24 0)
@@
     )
   )
-  (symbol (lib_id "Device:R") (at 261.62 148.59 90) (unit 1)
-    (in_bom yes) (on_board no) (dnp no)
-    (property "Reference" "R23" (at 261.62 146.05 90)
-      (effects (font (size 1.27 1.27)))
-    )
-    (property "Value" "100" (at 261.62 148.59 90)
-      (effects (font (size 1.27 1.27)))
-    )
-    (property "Footprint" "Resistor_THT:R_Axial_DIN0207_L6.3mm_D2.5mm_P10.16mm_Horizontal" (at 261.62 150.368 90)
-      (effects (font (size 1.27 1.27)) hide)
-    )
-    (property "Datasheet" "https://www.vishay.com/doc?31018" (at 261.62 148.59 0)
-      (effects (font (size 1.27 1.27)) hide)
-    )
-    (property "MPN" "CMF55100R00" (at 261.62 148.59 90)
-      (effects (font (size 1.27 1.27)) hide)
-    )
-    (pin "1")
-    (pin "2")
-    (instances
-      (project "OSDEHA_AMP"
-        (path "/59cc4414-299b-49db-9f9a-b06f69a12073"
-          (reference "R23") (unit 1)
-        )
-      )
-    )
-  )
   (symbol (lib_id "Device:R") (at 157.48 173.99 180) (unit 1)
     (in_bom yes) (on_board yes) (dnp no)
@@
         )
       )
-    )
-  )
-  (symbol (lib_id "Device:R") (at 308.61 148.59 90) (unit 1)
-    (in_bom yes) (on_board no) (dnp no)
-    (property "Reference" "R24" (at 308.61 146.05 90)
-      (effects (font (size 1.27 1.27)))
-    )
-    (property "Value" "100" (at 308.61 148.59 90)
-      (effects (font (size 1.27 1.27)))
-    )
-    (property "Footprint" "Resistor_THT:R_Axial_DIN0207_L6.3mm_D2.5mm_P10.16mm_Horizontal" (at 308.61 150.368 90)
-      (effects (font (size 1.27 1.27)) hide)
-    )
-    (property "Datasheet" "https://www.vishay.com/doc?31018" (at 308.61 148.59 0)
-      (effects (font (size 1.27 1.27)) hide)
-    )
-    (property "MPN" "CMF55100R00" (at 308.61 148.59 90)
-      (effects (font (size 1.27 1.27)) hide)
-    )
-    (pin "1")
-    (pin "2")
-    (instances
-      (project "OSDEHA_AMP"
-        (path "/59cc4414-299b-49db-9f9a-b06f69a12073"
-          (reference "R24") (unit 1)
-        )
-      )
