File: kicad/amplifier/OSDEHA_AMP.kicad_pcb (KiCad board)
At the start: 2 copper layers, 90 parts, among them J1 INPUT, J2 HEATERS DC, J3 PSU HV, J4 OUTPUT, J5 DHT FIL2, J6 DHT FIL1, Q1 DN2540N5-G, Q10 DN2540, Q2 DN2540N5-G, Q3 STF3LN80K5, Q4 STF3LN80K5, Q5 AOT1N60, Q6 IXTP3N100D2, Q7 AOT1N60, Q8 IXTP3N100D2, Q9 DN2540, SW1 SW_DPDT_x2, U1 6E5P, U2 6E5P, U3 801A, U4 801A

Commit message: HV filter caps
Parts:
- removed R25, R26, R29: 1M, Resistor_THT:R_Axial_DIN0207_L6.3mm_D2.5mm_P2.54mm_Vertical
- C5, C6, C7: value 51u -> 220n 630 V; footprint Capacitor_THT:CP_Radial_D25.0mm_P10.00mm_SnapIn -> Capacitor_THT:C_Rect_L18.0mm_W9.0mm_P15.00mm_FKS3_FKP3
- moved C7 62.8 mm to (250.7, 111.8)
- moved C6 34.2 mm to (250.7, 101.6)
- moved C5 13.1 mm to (250.7, 91.4)
- moved R44 13.0 mm to (216.8, 109.9)
- moved R45 13.0 mm to (219.1, 113.0)
- moved R46 13.0 mm to (217.2, 116.2)
- moved R47 13.0 mm to (229.9, 109.9)
- moved R48 13.0 mm to (227.6, 113.0)
- moved R49 13.0 mm to (229.6, 116.2)
- moved R27 13.0 mm to (227.6, 106.7)
- moved R28 13.0 mm to (219.1, 106.7)
- moved C9 3.89 mm to (235.8, 81.3)
- moved C3 0.78 mm to (157.9, 110.5)
- moved C2 0.60 mm to (157.9, 95.0)
Connections:
- C5 pad 1: /Dual_Gyrator/+HV -> GND
- C5 pad 2: GND -> /Dual_Gyrator/+HV

Commit message: PCB rearrange
Parts:
- R15, R20: footprint Resistor_THT:R_Axial_DIN0207_L6.3mm_D2.5mm_P2.54mm_Vertical -> Resistor_THT:R_Axial_DIN0207_L6.3mm_D2.5mm_P10.16mm_Horizontal
- moved C3 36.8 mm to (168.3, 75.2), turned to -90 degrees
- moved J4 33.9 mm to (192.3, 118.1)
- moved C2 31.6 mm to (133.3, 75.2), turned to -90 degrees
- moved R19 28.8 mm to (184.8, 101.0)
- moved R14 28.1 mm to (148.6, 101.0)
- moved C7 26.3 mm to (225.4, 104.5), turned to 90 degrees
- moved R18 25.3 mm to (188.6, 85.1), turned to 180 degrees
- moved R17 24.5 mm to (188.6, 89.5), turned to 180 degrees
- moved R16 24.2 mm to (188.6, 94.0), turned to 180 degrees
- moved R12 23.0 mm to (153.7, 90.2), turned to 180 degrees
- moved R27 22.5 mm to (211.0, 91.4)
- moved R48 22.5 mm to (211.0, 97.8)
- moved R49 22.5 mm to (213.1, 101.0)
- moved R47 22.5 mm to (213.4, 94.6)
- moved R13 22.5 mm to (153.7, 85.7), turned to 180 degrees
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
Commit message: pcb
Parts:
- removed H5: VENTILATION, MountingHole:MountingHole_5mm
- moved H4 222.6 mm to (251.5, 116.8)
- moved H3 193.8 mm to (225.4, 67.9)
- moved H1 64.9 mm to (95.2, 70.9)
- moved H2 64.4 mm to (70.5, 116.8)
- moved J2 9.65 mm to (125.1, 114.8)
- moved J3 7.86 mm to (241.5, 114.8)
- moved J5 3.90 mm to (203.2, 114.8)
- moved U4 3.89 mm to (221.5, 114.8)
- moved J6 3.81 mm to (159.7, 114.8)
- moved U3 3.81 mm to (177.7, 114.8)
- moved J4 3.80 mm to (190.3, 114.8)
- moved R7 3.42 mm to (79.1, 109.2)
- moved J1 3.29 mm to (97.2, 114.8)
- moved R1 2.96 mm to (111.5, 119.4)
- moved R3 2.29 mm to (85.1, 119.4)
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Routing:
- removed copper zone on F.Cu, net GND
Other:
- board outline added: 189.9 x 72.4 mm

Commit message: pcb
Parts:
- moved R40 10.2 mm to (181.6, 57.8), turned to -90 degrees
- moved R42 10.2 mm to (146.8, 57.8), turned to -90 degrees
- moved R41 2.54 mm to (186.7, 67.9)
- moved Q9 2.54 mm to (181.6, 53.1)
- moved D4 1.40 mm to (164.3, 58.5)
- moved D6 1.40 mm to (172.0, 58.5)
- moved Q4 1.40 mm to (165.6, 53.1)
- moved R22 1.40 mm to (168.1, 68.0)
- moved Q8 1.28 mm to (230.4, 53.1)
- moved R39 1.28 mm to (227.8, 58.1)
- moved R35 1.28 mm to (242.4, 51.1)
- moved R36 1.28 mm to (242.4, 54.9)
- moved R37 1.28 mm to (242.4, 58.7)
- moved R43 0.52 mm to (151.9, 68.1)
- moved Q3 0.43 mm to (130.8, 53.1)
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Other:
- board size 189.9 x 72.4 mm -> 190.1 x 72.4 mm

Commit message: pcb
Parts:
- moved H3 26.3 mm to (251.7, 67.6)
- moved R38 17.0 mm to (235.5, 70.9), turned to 0 degrees
- moved R35 10.2 mm to (252.6, 51.1), turned to 180 degrees
- moved D10 8.86 mm to (232.2, 65.5)
- moved D9 8.63 mm to (232.2, 70.6)
- moved Q7 1.06 mm to (243.1, 65.3), turned to 180 degrees
Changed lines of the file:
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@@
   )
   (footprint "Diode_THT:D_DO-41_SOD81_P7.62mm_Horizontal" (layer "F.Cu")
-    (at 239.275 70.81 180)
+    (at 232.156 65.532 180)
     (descr "Diode, DO-41_SOD81 series, Axial, Horizontal, pin pitch=7.62mm, , length*diameter=5.2*2.7mm^2, , http://www.diodes.com/_files/packages/DO-41%20(Plastic).pdf")
     (tags "Diode DO-41_SOD81 series Axial Horizontal pin pitch 7.62mm  length 5.2mm diameter 2.7mm")
@@
   )
   (footprint "MountingHole:MountingHole_3.2mm_M3" (layer "F.Cu")
-    (at 225.425 67.945)
+    (at 251.714 67.564)
     (descr "Mounting Hole 3.2mm, no annular, M3")
     (tags "mounting hole 3.2mm no annular m3")
@@
   )
   (footprint "Package_TO_SOT_THT:TO-220-3_Vertical" (layer "F.Cu")
-    (at 244.045 65.786 -90)
+    (at 243.078 65.349 180)
     (descr "TO-220-3, Vertical, RM 2.54mm, see https://www.vishay.com/docs/66542/to-220-1.pdf")
     (tags "TO-220-3 Vertical RM 2.54mm")
@@
     (property "ki_keywords" "N-Channel Depletion-Mode MOSFET")
     (attr through_hole)
-    (fp_text reference "Q7" (at -3.556 -0.811 -180) (layer "F.SilkS")
-        (effects (font (size 1 1) (thickness 0.15)))
-    )
-    (fp_text value "AOT1N60" (at 2.54 2.5 90) (layer "F.Fab")
-        (effects (font (size 1 1) (thickness 0.15)))
-    )
-    (fp_text user "${REFERENCE}" (at 2.54 -4.27 90) (layer "F.Fab")
+    (fp_text reference "Q7" (at -3.556 -0.811 90) (layer "F.SilkS")
+        (effects (font (size 1 1) (thickness 0.15)))
+    )
+    (fp_text value "AOT1N60" (at 2.54 2.5) (layer "F.Fab")
+        (effects (font (size 1 1) (thickness 0.15)))
+    )
+    (fp_text user "${REFERENCE}" (at 2.54 -4.27) (layer "F.Fab")
         (effects (font (size 1 1) (thickness 0.15)))
     )
@@
     (fp_line (start 7.54 1.25) (end 7.54 -3.15)
       (stroke (width 0.1) (type solid)) (layer "F.Fab"))
-    (pad "1" thru_hole rect (at 0 0 270) (size 1.905 2) (drill 1.1) (layers "*.Cu" "*.Mask")
+    (pad "1" thru_hole rect (at 0 0 180) (size 1.905 2) (drill 1.1) (layers "*.Cu" "*.Mask")
       (net 31 "Net-(D9-K)") (pinfunction "G") (pintype "input"))
-    (pad "2" thru_hole oval (at 2.54 0 270) (size 1.905 2) (drill 1.1) (layers "*.Cu" "*.Mask")
+    (pad "2" thru_hole oval (at 2.54 0 180) (size 1.905 2) (drill 1.1) (layers "*.Cu" "*.Mask")
       (net 35 "Net-(Q7-D)") (pinfunction "D") (pintype "passive"))
-    (pad "3" thru_hole oval (at 5.08 0 270) (size 1.905 2) (drill 1.1) (layers "*.Cu" "*.Mask")
+    (pad "3" thru_hole oval (at 5.08 0 180) (size 1.905 2) (drill 1.1) (layers "*.Cu" "*.Mask")
       (net 17 "/Dual_Gyrator/MU_OUT2") (pinfunction "S") (pintype "passive"))
     (model "${KICAD6_3DMODEL_DIR}/Package_TO_SOT_THT.3dshapes/TO-220-3_Vertical.wrl"
@@
   )
   (footprint "Resistor_THT:R_Axial_DIN0207_L6.3mm_D2.5mm_P10.16mm_Horizontal" (layer "F.Cu")
-    (at 250.698 63.246 -90)
+    (at 235.458 70.866)
     (descr "Resistor, Axial_DIN0207 series, Axial, Horizontal, pin pitch=10.16mm, 0.25W = 1/4W, length*diameter=6.3*2.5mm^2, http://cdn-reichelt.de/documents/datenblatt/B400/1_4W%23YAG.pdf")
     (tags "Resistor Axial_DIN0207 series Axial Horizontal pin pitch 10.16mm 0.25W = 1/4W length 6.3mm diameter 2.5mm")
@@
     (property "ki_keywords" "R res resistor")
     (attr through_hole)
-    (fp_text reference "R38" (at 5.08 -2.37 90) (layer "F.SilkS")
-        (effects (font (size 1 1) (thickness 0.15)))
-    )
-    (fp_text value "470" (at 5.08 2.37 90) (layer "F.Fab")
-        (effects (font (size 1 1) (thickness 0.15)))
-    )
-    (fp_text user "${REFERENCE}" (at 5.08 0 90) (layer "F.Fab")
+    (fp_text reference "R38" (at 5.08 -2.37) (layer "F.SilkS")
+        (effects (font (size 1 1) (thickness 0.15)))
+    )
+    (fp_text value "470" (at 5.08 2.37) (layer "F.Fab")
+        (effects (font (size 1 1) (thickness 0.15)))
+    )
+    (fp_text user "${REFERENCE}" (at 5.08 0) (layer "F.Fab")
         (effects (font (size 1 1) (thickness 0.15)))
     )
@@
     (fp_line (start 10.16 0) (end 8.23 0)
       (stroke (width 0.1) (type solid)) (layer "F.Fab"))
-    (pad "1" thru_hole circle (at 0 0 270) (size 1.6 1.6) (drill 0.8) (layers "*.Cu" "*.Mask")
+    (pad "1" thru_hole circle (at 0 0) (size 1.6 1.6) (drill 0.8) (layers "*.Cu" "*.Mask")
       (net 17 "/Dual_Gyrator/MU_OUT2") (pintype "passive"))
-    (pad "2" thru_hole oval (at 10.16 0 270) (size 1.6 1.6) (drill 0.8) (layers "*.Cu" "*.Mask")
+    (pad "2" thru_hole oval (at 10.16 0) (size 1.6 1.6) (drill 0.8) (layers "*.Cu" "*.Mask")
       (net 12 "/Dual_Gyrator/ANODE2") (pintype "passive"))
     (model "${KICAD6_3DMODEL_DIR}/Resistor_THT.3dshapes/R_Axial_DIN0207_L6.3mm_D2.5mm_P10.16mm_Horizontal.wrl"
@@
   )
   (footprint "Resistor_THT:R_Axial_DIN0207_L6.3mm_D2.5mm_P10.16mm_Horizontal" (layer "F.Cu")
-    (at 242.443 51.125)
+    (at 252.603 51.054 180)
     (descr "Resistor, Axial_DIN0207 series, Axial, Horizontal, pin pitch=10.16mm, 0.25W = 1/4W, length*diameter=6.3*2.5mm^2, http://cdn-reichelt.de/documents/datenblatt/B400/1_4W%23YAG.pdf")
     (tags "Resistor Axial_DIN0207 series Axial Horizontal pin pitch 10.16mm 0.25W = 1/4W length 6.3mm diameter 2.5mm")
@@
     (property "ki_keywords" "R res resistor")
     (attr through_hole)
-    (fp_text reference "R35" (at -1.785 -0.071 90) (layer "F.SilkS")
+    (fp_text reference "R35" (at 11.945 -0.071 90) (layer "F.SilkS")
         (effects (font (size 1 1) (thickness 0.15)))
     )
@@
     (fp_line (start 10.16 0) (end 8.23 0)
       (stroke (width 0.1) (type solid)) (layer "F.Fab"))
-    (pad "1" thru_hole circle (at 0 0) (size 1.6 1.6) (drill 0.8) (layers "*.Cu" "*.Mask")
+    (pad "1" thru_hole circle (at 0 0 180) (size 1.6 1.6) (drill 0.8) (layers "*.Cu" "*.Mask")
       (net 63 "Net-(R35-Pad1)") (pintype "passive"))
-    (pad "2" thru_hole oval (at 10.16 0) (size 1.6 1.6) (drill 0.8) (layers "*.Cu" "*.Mask")
+    (pad "2" thru_hole oval (at 10.16 0 180) (size 1.6 1.6) (drill 0.8) (layers "*.Cu" "*.Mask")
       (net 19 "GND") (pintype "passive"))
     (model "${KICAD6_3DMODEL_DIR}/Resistor_THT.3dshapes/R_Axial_DIN0207_L6.3mm_D2.5mm_P10.16mm_Horizontal.wrl"
@@
   )
   (footprint "Diode_THT:D_DO-41_SOD81_P7.62mm_Horizontal" (layer "F.Cu")
-    (at 239.275 65.73 180)
+    (at 232.156 70.612 180)
     (descr "Diode, DO-41_SOD81 series, Axial, Horizontal, pin pitch=7.62mm, , length*diameter=5.2*2.7mm^2, , http://www.diodes.com/_files/packages/DO-41%20(Plastic).pdf")
     (tags "Diode DO-41_SOD81 series Axial Horizontal pin pitch 7.62mm  length 5.2mm diameter 2.7mm")

Commit message: pcb
Parts:
- moved R38 17.7 mm to (251.5, 63.2), turned to -90 degrees
- moved H3 16.8 mm to (268.5, 66.3)
- moved R30 10.2 mm to (222.2, 51.1), turned to 180 degrees
- moved D10 6.98 mm to (236.7, 70.8)
- moved D9 6.69 mm to (236.7, 65.7)
- moved R33 3.30 mm to (221.7, 63.2)
- moved H1 2.41 mm to (96.0, 73.2)
- moved Q7 0.79 mm to (242.4, 65.7), turned to -90 degrees
- moved R35 0.64 mm to (252.0, 51.1)
- moved R36 0.64 mm to (241.8, 54.9)
- moved R37 0.64 mm to (241.8, 58.7)
Connections:
- U1 pad 4: Net-(Q2-D) -> unconnected-(U1A-K-Pad4)
- U2 pad 4: Net-(Q2-D) -> unconnected-(U2A-K-Pad4)
Routing:
- net /Dual_Gyrator/+HV: track 0.00 -> 222.5 mm
- net Net-(J2-Pin_2): track 0.00 -> 111.4 mm
- net Net-(Q2-D): track 0.00 -> 106.7 mm
- net Net-(U2A-A): track 0.00 -> 100.5 mm
- net Net-(U1A-A): track 0.00 -> 97.7 mm
- net Net-(J3-Pin_3): track 0.00 -> 66.4 mm
- net /Buffer_CCS_load1/NEG: track 0.00 -> 60.9 mm
- net /Dual_Gyrator/MU_OUT1: track 0.00 -> 50.4 mm
- net Net-(J2-Pin_1): track 0.00 -> 49.8 mm
- net /Dual_Gyrator/MU_OUT2: track 0.00 -> 42.1 mm
- net Net-(C1-Pad1): track 0.00 -> 31.5 mm
- net Net-(D9-K): track 0.00 -> 31.1 mm
- net Net-(D7-K): track 0.00 -> 30.5 mm
- net Net-(Q5-D): track 0.00 -> 25.1 mm
- net Net-(R10-Pad1): track 0.00 -> 24.3 mm
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
Commit message: pcb
Parts:
- moved H3 74.2 mm to (194.3, 63.0)
- moved H4 1.02 mm to (252.5, 116.8)
- moved R44 0.52 mm to (202.1, 94.6)
- moved R46 0.52 mm to (202.1, 101.0)
- moved R27 0.44 mm to (211.4, 91.4)
- moved R48 0.44 mm to (211.4, 97.8)
- moved R28 0.07 mm to (204.7, 91.4)
- moved R45 0.07 mm to (204.7, 97.8)
Connections:
- U1 pad 1: Net-(J2-Pin_2) -> Net-(J2-Pin_1)
- U1 pad 6: Net-(J2-Pin_1) -> Net-(J2-Pin_2)
- U2 pad 1: Net-(J2-Pin_2) -> Net-(J2-Pin_1)
- U2 pad 6: Net-(J2-Pin_1) -> Net-(J2-Pin_2)
- U3 pad 3: Net-(U3-G) -> /Buffer_CCS_load1/POS
- U4 pad 3: Net-(U4-G) -> /Buffer_CCS_load2/POS
Routing:
- net /Buffer_CCS_load1/NEG: track 60.9 -> 239.2 mm
- net /Dual_Gyrator/ANODE2: track 0.00 -> 123.3 mm, vias 0 -> 1
- net Net-(J3-Pin_3): track 66.4 -> 184.1 mm, vias 0 -> 2
- net /Buffer_CCS_load2/POS: track 16.8 -> 111.0 mm
- net /Buffer_CCS_load1/POS: track 16.5 -> 93.4 mm
- net /Dual_Gyrator/ANODE1: track 6.02 -> 73.9 mm
- net Net-(J2-Pin_2): track 111.4 -> 48.1 mm
- net GND: track 0.00 -> 57.4 mm, vias 0 -> 3
- net Net-(J2-Pin_1): track 49.8 -> 98.4 mm
- net /Dual_Gyrator/+HV: track 222.5 -> 252.3 mm
- net Net-(J4-Pin_1): track 0.00 -> 29.6 mm
- net Net-(J4-Pin_2): track 0.00 -> 27.9 mm
- net Net-(SW1B-B): track 0.00 -> 24.0 mm
- net Net-(Q7-D): track 0.00 -> 23.9 mm
- net Net-(SW1A-B): track 0.00 -> 23.0 mm
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- added copper zone on F.Cu, net GND

Commit message: pcb
Parts:
- moved R40 34.8 mm to (146.8, 57.9)
- moved R41 34.8 mm to (151.9, 68.1)
- moved R42 34.8 mm to (181.6, 57.9)
- moved Q10 34.8 mm to (181.6, 53.1)
- moved Q9 34.8 mm to (146.8, 53.1)
- moved R43 34.8 mm to (186.7, 68.1)
Connections:
- C1 pad 2: Net-(J3-Pin_3) -> /Buffer_CCS_load1/NEG
- C4 pad 2: Net-(J3-Pin_3) -> /Buffer_CCS_load1/NEG
- C6 pad 2: Net-(J3-Pin_3) -> /Buffer_CCS_load1/NEG
- C7 pad 2: /Buffer_CCS_load1/NEG -> Net-(J3-Pin_4)
- D5 pad 1: /Buffer_CCS_load1/POS -> /Buffer_CCS_load2/POS
- D6 pad 1: /Buffer_CCS_load2/POS -> /Buffer_CCS_load1/POS
- J3 pad 3: Net-(J3-Pin_3) -> /Buffer_CCS_load1/NEG
- J3 pad 4: /Buffer_CCS_load1/NEG -> Net-(J3-Pin_4)
- J5 pad 2: Net-(J3-Pin_3) -> /Buffer_CCS_load1/NEG
- J6 pad 2: Net-(J3-Pin_3) -> /Buffer_CCS_load1/NEG
- Q3 pad 3: /Buffer_CCS_load1/POS -> /Buffer_CCS_load2/POS
- Q4 pad 3: /Buffer_CCS_load2/POS -> /Buffer_CCS_load1/POS
- R10 pad 2: Net-(J3-Pin_3) -> /Buffer_CCS_load1/NEG
- R11 pad 2: /Buffer_CCS_load1/NEG -> Net-(J3-Pin_4)
- R12 pad 1: /Buffer_CCS_load1/NEG -> Net-(J3-Pin_4)
- R15 pad 1: Net-(J3-Pin_3) -> /Buffer_CCS_load1/NEG
- R16 pad 2: /Buffer_CCS_load1/NEG -> Net-(J3-Pin_4)
- R17 pad 1: /Buffer_CCS_load1/NEG -> Net-(J3-Pin_4)
- R20 pad 1: Net-(J3-Pin_3) -> /Buffer_CCS_load1/NEG
- U3 pad 1: Net-(J3-Pin_3) -> /Buffer_CCS_load1/NEG
- U3 pad 3: /Buffer_CCS_load1/POS -> /Buffer_CCS_load2/POS
- U4 pad 1: Net-(J3-Pin_3) -> /Buffer_CCS_load1/NEG
- U4 pad 3: /Buffer_CCS_load2/POS -> /Buffer_CCS_load1/POS
Routing:
- net Net-(J3-Pin_3): track 184.1 -> 0.00 mm, vias 2 -> 0
- net Net-(J3-Pin_4): track 0.00 -> 183.6 mm
- net GND: track 57.4 -> 99.4 mm, vias 3 -> 5
- net /Buffer_CCS_load1/NEG: track 239.2 -> 280.5 mm, vias 0 -> 2
- net /Buffer_CCS_load2/POS: track 111.0 -> 93.4 mm
- net /Buffer_CCS_load1/POS: track 93.4 -> 111.0 mm
- net Net-(D3-A): track 0.00 -> 8.41 mm
- net Net-(D10-A): track 0.00 -> 5.08 mm
- net /Dual_Gyrator/MU_OUT2: track 55.0 -> 59.1 mm
- net /Dual_Gyrator/ANODE2: track 123.3 -> 123.6 mm, vias 1 -> 2
