File: kicad/amplifier/OSDEHA_AMP.kicad_pcb (KiCad board)
At the start: 2 copper layers, 190.1 x 71.6 mm, 87 parts, among them J1 INPUT, J2 HEATERS DC, J3 PSU HV, J4 OUTPUT, J5 DHT FIL, Q1 DN2540, Q10 DN2540, Q2 DN2540, Q3 STF3LN80K5, Q4 STF3LN80K5, Q5 AOT1N60, Q6 IXTP3N100D2, Q7 AOT1N60, Q8 IXTP3N100D2, Q9 DN2540, SW1 SW_DPDT_x2, U1 6E5P, U2 6E5P, U3 801A, U4 801A

Commit message: add Zener clamp to DHT grids to prevent too much positive grid voltage
Parts:
- R34, R39, R40, R42, R5, R8: value 300 -> 1k
Connections:
- D5 pad 1: /G1 -> /Buffer_CCS_load2/POS
- D6 pad 1: /G2 -> /Buffer_CCS_load1/POS
- Q10 pad 2: /G2 -> /Buffer_CCS_load1/POS
- Q3 pad 3: /G1 -> /Buffer_CCS_load2/POS
- Q4 pad 3: /G2 -> /Buffer_CCS_load1/POS
- Q9 pad 2: /G1 -> /Buffer_CCS_load2/POS
Changed lines of the file:
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@@
 	(net 71 "Net-(Q5-G)")
 	(net 72 "Net-(Q7-G)")
+	(net 73 "/Buffer_CCS_load2/POS")
+	(net 74 "/Buffer_CCS_load1/POS")
 	(footprint "Resistor_THT:R_Axial_DIN0207_L6.3mm_D2.5mm_P10.16mm_Horizontal"
 		(layer "F.Cu")
@@
 			(layers "*.Cu" "*.Mask")
 			(remove_unused_layers no)
-			(net 63 "/G1")
+			(net 73 "/Buffer_CCS_load2/POS")
 			(pinfunction "S")
 			(pintype "passive")
@@
 			(layers "*.Cu" "*.Mask")
 			(remove_unused_layers no)
-			(net 64 "/G2")
+			(net 74 "/Buffer_CCS_load1/POS")
 			(pinfunction "D")
 			(pintype "passive")
@@
 			)
 		)
-		(property "Value" "300"
+		(property "Value" "1k"
 			(at 5.08 2.37 90)
 			(layer "F.Fab")
@@
 			)
 		)
-		(property "MPN" "CMF55300R00"
+		(property "MPN" "CMF551K000"
 			(at 0 0 0)
 			(layer "F.Fab")
@@
 			)
 		)
-		(property "Value" "300"
+		(property "Value" "1k"
 			(at 5.08 2.37 90)
 			(layer "F.Fab")
@@
 			)
 		)
-		(property "MPN" "CMF55300R00"
+		(property "MPN" "CMF551K000"
 			(at 0 0 0)
 			(layer "F.Fab")
@@
 			(layers "*.Cu" "*.Mask")
 			(remove_unused_layers no)
-			(net 64 "/G2")
+			(net 74 "/Buffer_CCS_load1/POS")
 			(pinfunction "K")
 			(pintype "passive")
@@
 			)
 		)
-		(property "Value" "300"
+		(property "Value" "1k"
 			(at 5.08 2.37 0)
 			(layer "F.Fab")
@@
 			)
 		)
-		(property "MPN" "CMF55300R00"
+		(property "MPN" "CMF551K000"
 			(at 0 0 0)
 			(layer "F.Fab")
@@
 			(layers "*.Cu" "*.Mask")
 			(remove_unused_layers no)
-			(net 63 "/G1")
+			(net 73 "/Buffer_CCS_load2/POS")
 			(pinfunction "D")
 			(pintype "passive")
@@
 		(tags "Resistor Axial_DIN0516 series Axial Vertical pin pitch 5.08mm 2W length 15.5mm diameter 5mm")
 		(property "Reference" "R33"
-			(at 4.78 2.875 270)
+			(at 4.78 2.875 -90)
 			(layer "F.SilkS")
 			(effects
@@
 		)
 		(property "Value" "470"
-			(at 2.54 3.62 270)
+			(at 2.54 3.62 -90)
 			(layer "F.Fab")
 			(hide yes)
@@
 		)
 		(fp_text user "${REFERENCE}"
-			(at 2.54 -3.62 270)
+			(at 2.54 -3.62 -90)
 			(layer "F.Fab")
 			(effects
@@
 			)
 		)
-		(property "Value" "300"
+		(property "Value" "1k"
 			(at 5.08 2.37 0)
 			(layer "F.Fab")
@@
 			)
 		)
-		(property "MPN" "CMF55300R00"
+		(property "MPN" "CMF551K000"
 			(at 0 0 0)
 			(layer "F.Fab")
@@
 			)
 		)
-		(property "Value" "300"
+		(property "Value" "1k"
 			(at 5.08 2.37 90)
 			(layer "F.Fab")
@@
 			)
 		)
-		(property "MPN" "CMF55300R00"
+		(property "MPN" "CMF551K000"
 			(at 0 0 0)
 			(layer "F.Fab")
@@
 			)
 		)
-		(property "Value" "300"
+		(property "Value" "1k"
 			(at 5.08 2.37 0)
 			(layer "F.Fab")
@@
 			)
 		)
-		(property "MPN" "CMF55300R00"
+		(property "MPN" "CMF551K000"
 			(at 0 0 0)
 			(layer "F.Fab")
@@
 			(layers "*.Cu" "*.Mask")
 			(remove_unused_layers no)
-			(net 63 "/G1")
+			(net 73 "/Buffer_CCS_load2/POS")
 			(pinfunction "K")
 			(pintype "passive")
@@
 			(layers "*.Cu" "*.Mask")
 			(remove_unused_layers no)
-			(net 64 "/G2")
+			(net 74 "/Buffer_CCS_load1/POS")
 			(pinfunction "S")
 			(pintype "passive")

Commit message: revise diode clamp at DHT grids
Connections:
- D5 pad 1: /Buffer_CCS_load2/POS -> /G1
- D6 pad 1: /Buffer_CCS_load1/POS -> /G2
- Q10 pad 2: /Buffer_CCS_load1/POS -> /G2
- Q3 pad 3: /Buffer_CCS_load2/POS -> /G1
- Q4 pad 3: /Buffer_CCS_load1/POS -> /G2
- Q9 pad 2: /Buffer_CCS_load2/POS -> /G1
- U3 pad 3: /G1 -> Net-(U3-G)
- U4 pad 3: /G2 -> Net-(U4-G)
Changed lines of the file:
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@@
 	(net 71 "Net-(Q5-G)")
 	(net 72 "Net-(Q7-G)")
-	(net 73 "/Buffer_CCS_load2/POS")
-	(net 74 "/Buffer_CCS_load1/POS")
+	(net 73 "Net-(U3-G)")
+	(net 74 "Net-(U4-G)")
 	(footprint "Resistor_THT:R_Axial_DIN0207_L6.3mm_D2.5mm_P10.16mm_Horizontal"
 		(layer "F.Cu")
@@
 			(layers "*.Cu" "*.Mask")
 			(remove_unused_layers no)
-			(net 73 "/Buffer_CCS_load2/POS")
+			(net 63 "/G1")
 			(pinfunction "S")
 			(pintype "passive")
@@
 			(layers "*.Cu" "*.Mask")
 			(remove_unused_layers no)
-			(net 74 "/Buffer_CCS_load1/POS")
+			(net 64 "/G2")
 			(pinfunction "D")
 			(pintype "passive")
@@
 			(layers "*.Cu" "*.Mask")
 			(remove_unused_layers no)
-			(net 74 "/Buffer_CCS_load1/POS")
+			(net 64 "/G2")
 			(pinfunction "K")
 			(pintype "passive")
@@
 			(layers "*.Cu" "*.Mask")
 			(remove_unused_layers no)
-			(net 73 "/Buffer_CCS_load2/POS")
+			(net 63 "/G1")
 			(pinfunction "D")
 			(pintype "passive")
@@
 			(layers "*.Cu" "*.Mask")
 			(remove_unused_layers no)
-			(net 63 "/G1")
+			(net 73 "Net-(U3-G)")
 			(pinfunction "G")
 			(pintype "input")
@@
 			(layers "*.Cu" "*.Mask")
 			(remove_unused_layers no)
-			(net 73 "/Buffer_CCS_load2/POS")
+			(net 63 "/G1")
 			(pinfunction "K")
 			(pintype "passive")
@@
 			(layers "*.Cu" "*.Mask")
 			(remove_unused_layers no)
-			(net 64 "/G2")
+			(net 74 "Net-(U4-G)")
 			(pinfunction "G")
 			(pintype "input")
@@
 			(layers "*.Cu" "*.Mask")
 			(remove_unused_layers no)
-			(net 74 "/Buffer_CCS_load1/POS")
+			(net 64 "/G2")
 			(pinfunction "S")
 			(pintype "passive")
