File: kicad/powersupply_colemanreg/COLEMAN_RAW_DC.kicad_sch (KiCad schematic)
At the start: 9 parts

Commit message: psu
Parts:
- renumbered C15 to C1, C16 to C2, D24 to D1, D25 to D2, D26 to D3, D27 to D4, R34 to R1, R35 to R2, R36 to R3
Changed lines of the file:
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@@
   (symbol (lib_id "Diode:1N5822") (at 91.44 82.55 270) (unit 1)
     (in_bom yes) (on_board yes) (dnp no) (fields_autoplaced)
-    (property "Reference" "D27" (at 93.98 80.9625 90)
+    (property "Reference" "D4" (at 93.98 80.9625 90)
       (effects (font (size 1.27 1.27)) (justify left))
     )
@@
     (pin "1")
     (instances
-      (project "powersupply_colemanreg"
-        (path "/6a766a35-7f7e-4680-bf64-1ed131aec470/5c8de33b-0aec-4bd3-8a06-d4311bc9100c"
-          (reference "D27") (unit 1)
-        )
-        (path "/6a766a35-7f7e-4680-bf64-1ed131aec470/a7689cda-8b81-433b-9126-0f3438ec2ce2"
-          (reference "D27") (unit 1)
+      (project "OSDEHA_powersupply_colemanreg"
+        (path "/6a766a35-7f7e-4680-bf64-1ed131aec470/5c8de33b-0aec-4bd3-8a06-d4311bc9100c"
+          (reference "D4") (unit 1)
+        )
+        (path "/6a766a35-7f7e-4680-bf64-1ed131aec470/a7689cda-8b81-433b-9126-0f3438ec2ce2"
+          (reference "D8") (unit 1)
         )
       )
@@
   (symbol (lib_id "Diode:1N5822") (at 76.2 82.55 270) (unit 1)
     (in_bom yes) (on_board yes) (dnp no) (fields_autoplaced)
-    (property "Reference" "D25" (at 78.74 80.9625 90)
+    (property "Reference" "D2" (at 78.74 80.9625 90)
       (effects (font (size 1.27 1.27)) (justify left))
     )
@@
     (pin "1")
     (instances
-      (project "powersupply_colemanreg"
-        (path "/6a766a35-7f7e-4680-bf64-1ed131aec470/5c8de33b-0aec-4bd3-8a06-d4311bc9100c"
-          (reference "D25") (unit 1)
-        )
-        (path "/6a766a35-7f7e-4680-bf64-1ed131aec470/a7689cda-8b81-433b-9126-0f3438ec2ce2"
-          (reference "D25") (unit 1)
+      (project "OSDEHA_powersupply_colemanreg"
+        (path "/6a766a35-7f7e-4680-bf64-1ed131aec470/5c8de33b-0aec-4bd3-8a06-d4311bc9100c"
+          (reference "D2") (unit 1)
+        )
+        (path "/6a766a35-7f7e-4680-bf64-1ed131aec470/a7689cda-8b81-433b-9126-0f3438ec2ce2"
+          (reference "D6") (unit 1)
         )
       )
@@
   (symbol (lib_id "Device:R") (at 130.81 87.63 90) (unit 1)
     (in_bom yes) (on_board yes) (dnp no)
-    (property "Reference" "R36" (at 130.81 85.09 90)
+    (property "Reference" "R3" (at 130.81 85.09 90)
       (effects (font (size 1.27 1.27)))
     )
@@
     (pin "2")
     (instances
-      (project "powersupply_colemanreg"
-        (path "/6a766a35-7f7e-4680-bf64-1ed131aec470/5c8de33b-0aec-4bd3-8a06-d4311bc9100c"
-          (reference "R36") (unit 1)
-        )
-        (path "/6a766a35-7f7e-4680-bf64-1ed131aec470/a7689cda-8b81-433b-9126-0f3438ec2ce2"
-          (reference "R36") (unit 1)
+      (project "OSDEHA_powersupply_colemanreg"
+        (path "/6a766a35-7f7e-4680-bf64-1ed131aec470/5c8de33b-0aec-4bd3-8a06-d4311bc9100c"
+          (reference "R3") (unit 1)
+        )
+        (path "/6a766a35-7f7e-4680-bf64-1ed131aec470/a7689cda-8b81-433b-9126-0f3438ec2ce2"
+          (reference "R6") (unit 1)
         )
       )
@@
   (symbol (lib_id "Diode:1N5822") (at 91.44 67.31 270) (unit 1)
     (in_bom yes) (on_board yes) (dnp no) (fields_autoplaced)
-    (property "Reference" "D26" (at 93.98 65.7225 90)
+    (property "Reference" "D3" (at 93.98 65.7225 90)
       (effects (font (size 1.27 1.27)) (justify left))
     )
@@
     (pin "1")
     (instances
-      (project "powersupply_colemanreg"
-        (path "/6a766a35-7f7e-4680-bf64-1ed131aec470/5c8de33b-0aec-4bd3-8a06-d4311bc9100c"
-          (reference "D26") (unit 1)
-        )
-        (path "/6a766a35-7f7e-4680-bf64-1ed131aec470/a7689cda-8b81-433b-9126-0f3438ec2ce2"
-          (reference "D26") (unit 1)
+      (project "OSDEHA_powersupply_colemanreg"
+        (path "/6a766a35-7f7e-4680-bf64-1ed131aec470/5c8de33b-0aec-4bd3-8a06-d4311bc9100c"
+          (reference "D3") (unit 1)
+        )
+        (path "/6a766a35-7f7e-4680-bf64-1ed131aec470/a7689cda-8b81-433b-9126-0f3438ec2ce2"
+          (reference "D7") (unit 1)
         )
       )
@@
   (symbol (lib_id "Diode:1N5822") (at 76.2 67.31 270) (unit 1)
     (in_bom yes) (on_board yes) (dnp no) (fields_autoplaced)
-    (property "Reference" "D24" (at 78.74 65.7225 90)
+    (property "Reference" "D1" (at 78.74 65.7225 90)
       (effects (font (size 1.27 1.27)) (justify left))
     )
@@
     (pin "1")
     (instances
-      (project "powersupply_colemanreg"
-        (path "/6a766a35-7f7e-4680-bf64-1ed131aec470/5c8de33b-0aec-4bd3-8a06-d4311bc9100c"
-          (reference "D24") (unit 1)
-        )
-        (path "/6a766a35-7f7e-4680-bf64-1ed131aec470/a7689cda-8b81-433b-9126-0f3438ec2ce2"
-          (reference "D24") (unit 1)
+      (project "OSDEHA_powersupply_colemanreg"
+        (path "/6a766a35-7f7e-4680-bf64-1ed131aec470/5c8de33b-0aec-4bd3-8a06-d4311bc9100c"
+          (reference "D1") (unit 1)
+        )
+        (path "/6a766a35-7f7e-4680-bf64-1ed131aec470/a7689cda-8b81-433b-9126-0f3438ec2ce2"
+          (reference "D5") (unit 1)
         )
       )
@@
   (symbol (lib_id "Device:C_Polarized") (at 121.92 74.93 0) (unit 1)
     (in_bom yes) (on_board yes) (dnp no)
-    (property "Reference" "C15" (at 123.19 72.39 0)
+    (property "Reference" "C1" (at 123.19 72.39 0)
       (effects (font (size 1.27 1.27)) (justify left))
     )
@@
     (pin "2")
     (instances
-      (project "powersupply_colemanreg"
-        (path "/6a766a35-7f7e-4680-bf64-1ed131aec470/5c8de33b-0aec-4bd3-8a06-d4311bc9100c"
-          (reference "C15") (unit 1)
-        )
-        (path "/6a766a35-7f7e-4680-bf64-1ed131aec470/a7689cda-8b81-433b-9126-0f3438ec2ce2"
-          (reference "C15") (unit 1)
+      (project "OSDEHA_powersupply_colemanreg"
+        (path "/6a766a35-7f7e-4680-bf64-1ed131aec470/5c8de33b-0aec-4bd3-8a06-d4311bc9100c"
+          (reference "C1") (unit 1)
+        )
+        (path "/6a766a35-7f7e-4680-bf64-1ed131aec470/a7689cda-8b81-433b-9126-0f3438ec2ce2"
+          (reference "C3") (unit 1)
         )
       )
@@
   (symbol (lib_id "Device:C_Polarized") (at 139.7 74.93 0) (unit 1)
     (in_bom yes) (on_board yes) (dnp no)
-    (property "Reference" "C16" (at 140.97 72.39 0)
+    (property "Reference" "C2" (at 140.97 72.39 0)
       (effects (font (size 1.27 1.27)) (justify left))
     )
@@
     (pin "2")
     (instances
-      (project "powersupply_colemanreg"
-        (path "/6a766a35-7f7e-4680-bf64-1ed131aec470/5c8de33b-0aec-4bd3-8a06-d4311bc9100c"
-          (reference "C16") (unit 1)
-        )
-        (path "/6a766a35-7f7e-4680-bf64-1ed131aec470/a7689cda-8b81-433b-9126-0f3438ec2ce2"
-          (reference "C16") (unit 1)
+      (project "OSDEHA_powersupply_colemanreg"
+        (path "/6a766a35-7f7e-4680-bf64-1ed131aec470/5c8de33b-0aec-4bd3-8a06-d4311bc9100c"
+          (reference "C2") (unit 1)
+        )
+        (path "/6a766a35-7f7e-4680-bf64-1ed131aec470/a7689cda-8b81-433b-9126-0f3438ec2ce2"
+          (reference "C4") (unit 1)
         )
       )
@@
   (symbol (lib_id "Device:R") (at 106.68 74.93 0) (unit 1)
     (in_bom yes) (on_board yes) (dnp no)
-    (property "Reference" "R34" (at 104.14 71.12 0)
+    (property "Reference" "R1" (at 104.14 71.12 0)
       (effects (font (size 1.27 1.27)))
     )
@@
     (pin "2")
     (instances
-      (project "powersupply_colemanreg"
-        (path "/6a766a35-7f7e-4680-bf64-1ed131aec470/5c8de33b-0aec-4bd3-8a06-d4311bc9100c"
-          (reference "R34") (unit 1)
-        )
-        (path "/6a766a35-7f7e-4680-bf64-1ed131aec470/a7689cda-8b81-433b-9126-0f3438ec2ce2"
-          (reference "R34") (unit 1)
+      (project "OSDEHA_powersupply_colemanreg"
+        (path "/6a766a35-7f7e-4680-bf64-1ed131aec470/5c8de33b-0aec-4bd3-8a06-d4311bc9100c"
+          (reference "R1") (unit 1)
+        )
+        (path "/6a766a35-7f7e-4680-bf64-1ed131aec470/a7689cda-8b81-433b-9126-0f3438ec2ce2"
+          (reference "R4") (unit 1)
         )
       )
@@
   (symbol (lib_id "Device:R") (at 130.81 62.23 90) (unit 1)
     (in_bom yes) (on_board yes) (dnp no)
-    (property "Reference" "R35" (at 130.81 59.69 90)
+    (property "Reference" "R2" (at 130.81 59.69 90)
       (effects (font (size 1.27 1.27)))
     )
@@
     (pin "2")
     (instances
-      (project "powersupply_colemanreg"
-        (path "/6a766a35-7f7e-4680-bf64-1ed131aec470/5c8de33b-0aec-4bd3-8a06-d4311bc9100c"
-          (reference "R35") (unit 1)
-        )
-        (path "/6a766a35-7f7e-4680-bf64-1ed131aec470/a7689cda-8b81-433b-9126-0f3438ec2ce2"
-          (reference "R35") (unit 1)
-        )
-      )
+      (project "OSDEHA_powersupply_colemanreg"
+        (path "/6a766a35-7f7e-4680-bf64-1ed131aec470/5c8de33b-0aec-4bd3-8a06-d4311bc9100c"
+          (reference "R2") (unit 1)
+        )
+        (path "/6a766a35-7f7e-4680-bf64-1ed131aec470/a7689cda-8b81-433b-9126-0f3438ec2ce2"
+          (reference "R5") (unit 1)
+        )
+      )
