File: kicad/powersupply_colemanreg/OSDEHA_powersupply_colemanreg.kicad_sch (KiCad schematic)
At the start: 6 parts, among them J1 10.5 VAC / 4.5 A, J2 10.5 VAC / 4.5 A, J3 COLEMANREG-LEFT-1, J4 COLEMANREG-LEFT-2, J5 COLEMANREG-RIGHT-1, J6 COLEMANREG-RIGHT-2

Commit message: cleanup
Other:
- note added: "Each channel has two Coleman DHT filament regulators, which share a common raw DC supply. Raw DC supplies must be floating! The DHT regs are referenced to the respective B- rail on the amplifier boards. Raw DC supplies must use separate AC windings!"
- note removed: "Each channel has two Coleman DHT filament regulators, which share a common raw DW supply. Raw DC supplies must be floating! The DHT regs are referenced to the respective B- rail on the amplifier boards. Raw DC supplies must use separate AC windings!"
Changed lines of the file:
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@@
     (effects (font (size 1.27 1.27)) (justify left bottom))
   )
-  (text "Each channel has two Coleman DHT filament regulators, which share a common raw DW supply.\nRaw DC supplies must be floating! The DHT regs are referenced to the respective B- rail on the amplifier boards.\nRaw DC supplies must use separate AC windings!"
+  (text "Each channel has two Coleman DHT filament regulators, which share a common raw DC supply.\nRaw DC supplies must be floating! The DHT regs are referenced to the respective B- rail on the amplifier boards.\nRaw DC supplies must use separate AC windings!"
     (at 38.1 53.34 0)
     (effects (font (size 1.27 1.27)) (justify left bottom))
