File: kicad/powersupply/OSDEHA_PSU.kicad_pcb (KiCad board)
At the start: 2 copper layers, 128 parts, among them J1 340 VAC / 220 mA, J10 HEATERS-LEFT, J11 HEATERS-RIGHT, J12 COLEMANREG-LEFT-1, J13 COLEMANREG-LEFT-2, J14 COLEMANREG-RIGHT-1, J15 COLEMANREG-RIGHT-2, J2 340 VAC / 220 mA, J3 420 VAC / 75 mA, J4 9 VAC / 4.5 A, J5 10.5 VAC / 4.5 A, J6 10.5 VAC / 4.5 A, J7 Stator bias, J8 HV-L, J9 HV-R, K1 RT424006, Q1 BD138, Q10 BC550, Q11 LND150, Q12 LND150, Q13 NTHL1000N170M1, Q14 BC550, Q2 10M90S, Q3 LND150, Q4 LND150, Q5 NTHL1000N170M1, Q6 BC550, Q7 LND150, Q8 LND150, Q9 NTHL1000N170M1, U1 LM1085-ADJ, U2 NE555P

Commit message: psu
Parts:
- C7: value 10u 16 V -> 22u 16 V
- D5, D7: footprint Diode_THT:D_DO-41_SOD81_P10.16mm_Horizontal -> Diode_THT:D_DO-41_SOD81_P7.62mm_Horizontal
- R12, R13, R4: footprint Resistor_THT:R_Axial_DIN0207_L6.3mm_D2.5mm_P10.16mm_Horizontal -> Resistor_THT:R_Axial_DIN0207_L6.3mm_D2.5mm_P2.54mm_Vertical
- moved D25 316.9 mm to (250.4, 97.0)
- moved D26 316.9 mm to (250.4, 101.2)
- moved J4 311.2 mm to (-18.5, 220.3)
- moved J11 296.6 mm to (-9.07, 206.5)
- moved D27 291.6 mm to (249.7, 138.6)
- moved D28 291.6 mm to (256.7, 136.0)
- moved R34 263.9 mm to (159.8, 72.6)
- moved D24 260.3 mm to (227.8, 89.5)
- moved R15 259.4 mm to (-65.4, 210.9), turned to 90 degrees
- moved D2 247.3 mm to (-31.3, 222.5), turned to 90 degrees
- moved D4 247.1 mm to (-44.8, 222.5), turned to 90 degrees
- moved J10 245.8 mm to (-19.6, 206.5), turned to 180 degrees
- moved D1 244.9 mm to (-26.3, 217.4), turned to -90 degrees
- moved D3 244.4 mm to (-39.8, 217.4), turned to -90 degrees
- moved U2 237.6 mm to (-40.9, 178.4), turned to 180 degrees
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
Commit message: up
Parts:
- moved J5 44.8 mm to (247.5, 28.1)
- moved D24 44.8 mm to (234.1, 45.2)
- moved D25 44.8 mm to (256.7, 52.6)
- moved D26 44.8 mm to (256.7, 56.9)
- moved D27 44.8 mm to (255.9, 94.2)
- moved D28 44.8 mm to (262.9, 91.7)
- moved D29 44.8 mm to (217.8, 64.9)
- moved R39 44.8 mm to (207.5, 49.4)
- moved H3 0.68 mm to (147.6, 170.7)
Other:
- board text added: "CHASSIS EARTH"
Changed lines of the file:
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@@
     (property "ki_keywords" "mounting hole")
     (attr exclude_from_pos_files)
-    (fp_text reference "CHASSIS1" (at 0 -4.2) (layer "F.SilkS")
+    (fp_text reference "CHASSIS1" (at 0 -4.2) (layer "F.SilkS") hide
         (effects (font (size 1 1) (thickness 0.15)))
     )
@@
   )
   (footprint "TerminalBlock_Phoenix:TerminalBlock_Phoenix_MKDS-1,5-2-5.08_1x02_P5.08mm_Horizontal" (layer "F.Cu")
-    (at 241.3 72.39)
+    (at 247.523 28.067)
     (descr "Terminal Block Phoenix MKDS-1,5-2-5.08, 2 pins, pitch 5.08mm, size 10.2x9.8mm^2, drill diamater 1.3mm, pad diameter 2.6mm, see http://www.farnell.com/datasheets/100425.pdf, script-generated using https://github.com/pointhi/kicad-footprint-generator/scripts/TerminalBlock_Phoenix")
     (tags "THT Terminal Block Phoenix MKDS-1,5-2-5.08 pitch 5.08mm size 10.2x9.8mm^2 drill 1.3mm pad 2.6mm")
@@
   )
   (footprint "Diode_THT:D_DO-201AD_P15.24mm_Horizontal" (layer "F.Cu")
-    (at 250.444 101.219)
+    (at 256.667 56.896)
     (descr "Diode, DO-201AD series, Axial, Horizontal, pin pitch=15.24mm, , length*diameter=9.5*5.2mm^2, , http://www.diodes.com/_files/packages/DO-201AD.pdf")
     (tags "Diode DO-201AD series Axial Horizontal pin pitch 15.24mm  length 9.5mm diameter 5.2mm")
@@
   )
   (footprint "Diode_THT:D_DO-201AD_P15.24mm_Horizontal" (layer "F.Cu")
-    (at 227.838 89.535)
+    (at 234.061 45.212)
     (descr "Diode, DO-201AD series, Axial, Horizontal, pin pitch=15.24mm, , length*diameter=9.5*5.2mm^2, , http://www.diodes.com/_files/packages/DO-201AD.pdf")
     (tags "Diode DO-201AD series Axial Horizontal pin pitch 15.24mm  length 9.5mm diameter 5.2mm")
@@
   )
   (footprint "Resistor_THT:R_Axial_DIN0614_L14.3mm_D5.7mm_P15.24mm_Horizontal" (layer "F.Cu")
-    (at 201.315 93.71)
+    (at 207.538 49.387)
     (descr "Resistor, Axial_DIN0614 series, Axial, Horizontal, pin pitch=15.24mm, 1.5W, length*diameter=14.3*5.7mm^2")
     (tags "Resistor Axial_DIN0614 series Axial Horizontal pin pitch 15.24mm 1.5W length 14.3mm diameter 5.7mm")
@@
     (property "ki_keywords" "mounting hole")
     (attr exclude_from_pos_files)
-    (fp_text reference "H2" (at 0 -4.2) (layer "F.SilkS")
+    (fp_text reference "H2" (at 0 -4.2) (layer "F.SilkS") hide
         (effects (font (size 1 1) (thickness 0.15)))
     )
@@
   )
   (footprint "Diode_THT:D_DO-201AD_P15.24mm_Horizontal" (layer "F.Cu")
-    (at 211.582 109.22)
+    (at 217.805 64.897)
     (descr "Diode, DO-201AD series, Axial, Horizontal, pin pitch=15.24mm, , length*diameter=9.5*5.2mm^2, , http://www.diodes.com/_files/packages/DO-201AD.pdf")
     (tags "Diode DO-201AD series Axial Horizontal pin pitch 15.24mm  length 9.5mm diameter 5.2mm")
@@
   )
   (footprint "Diode_THT:D_DO-201AD_P15.24mm_Horizontal" (layer "F.Cu")
-    (at 249.682 138.557 90)
+    (at 255.905 94.234 90)
     (descr "Diode, DO-201AD series, Axial, Horizontal, pin pitch=15.24mm, , length*diameter=9.5*5.2mm^2, , http://www.diodes.com/_files/packages/DO-201AD.pdf")
     (tags "Diode DO-201AD series Axial Horizontal pin pitch 15.24mm  length 9.5mm diameter 5.2mm")
@@
   )
   (footprint "MountingHole:MountingHole_3.2mm_M3" (layer "F.Cu")
-    (at 146.939 170.942)
+    (at 147.574 170.688)
     (descr "Mounting Hole 3.2mm, no annular, M3")
     (tags "mounting hole 3.2mm no annular m3")
@@
     (property "ki_keywords" "mounting hole")
     (attr exclude_from_pos_files)
-    (fp_text reference "H3" (at 0 -4.2) (layer "F.SilkS")
+    (fp_text reference "H3" (at 0 -4.2) (layer "F.SilkS") hide
         (effects (font (size 1 1) (thickness 0.15)))
     )
@@
   )
   (footprint "Diode_THT:D_DO-201AD_P15.24mm_Horizontal" (layer "F.Cu")
-    (at 256.667 136.017 -90)
+    (at 262.89 91.694 -90)
     (descr "Diode, DO-201AD series, Axial, Horizontal, pin pitch=15.24mm, , length*diameter=9.5*5.2mm^2, , http://www.diodes.com/_files/packages/DO-201AD.pdf")
     (tags "Diode DO-201AD series Axial Horizontal pin pitch 15.24mm  length 9.5mm diameter 5.2mm")
@@
     (property "ki_keywords" "mounting hole")
     (attr exclude_from_pos_files)
-    (fp_text reference "H1" (at 0 -4.2) (layer "F.SilkS")
+    (fp_text reference "H1" (at 0 -4.2) (layer "F.SilkS") hide
         (effects (font (size 1 1) (thickness 0.15)))
     )
@@
   )
   (footprint "Diode_THT:D_DO-201AD_P15.24mm_Horizontal" (layer "F.Cu")
-    (at 250.444 96.969)
+    (at 256.667 52.646)
     (descr "Diode, DO-201AD series, Axial, Horizontal, pin pitch=15.24mm, , length*diameter=9.5*5.2mm^2, , http://www.diodes.com/_files/packages/DO-201AD.pdf")
     (tags "Diode DO-201AD series Axial Horizontal pin pitch 15.24mm  length 9.5mm diameter 5.2mm")
@@
     )
   )
+  (gr_text "CHASSIS\nEARTH" (at -60.833 223.139) (layer "F.SilkS")
+    (effects (font (size 1.5 1.5) (thickness 0.3) bold) (justify left bottom))
+  )
 )

Commit message: psu
Parts:
- removed C15, C16, C17, C18: 15000u 25 V, Capacitor_THT:CP_Radial_D25.0mm_P10.00mm_SnapIn
- removed D24, D25, D26, D27, D28, D29, D30, D31: 1N5822, Diode_THT:D_DO-201AD_P15.24mm_Horizontal
- removed J10: HEATERS-LEFT, Connector_Molex:Molex_KK-396_A-41791-0002_1x02_P3.96mm_Vertical
- removed J11: HEATERS-RIGHT, Connector_Molex:Molex_KK-396_A-41791-0002_1x02_P3.96mm_Vertical
- removed J12: COLEMANREG-LEFT-1, Connector_Molex:Molex_KK-396_A-41791-0002_1x02_P3.96mm_Vertical
- removed J13: COLEMANREG-LEFT-2, Connector_Molex:Molex_KK-396_A-41791-0002_1x02_P3.96mm_Vertical
- removed J14: COLEMANREG-RIGHT-1, Connector_Molex:Molex_KK-396_A-41791-0002_1x02_P3.96mm_Vertical
- removed J15: COLEMANREG-RIGHT-2, Connector_Molex:Molex_KK-396_A-41791-0002_1x02_P3.96mm_Vertical
- removed R34, R37: 10k, Resistor_THT:R_Axial_DIN0207_L6.3mm_D2.5mm_P10.16mm_Horizontal
- removed R35, R36, R38, R39: 0.22 3 W, Resistor_THT:R_Axial_DIN0614_L14.3mm_D5.7mm_P15.24mm_Horizontal
- J5: value 10.5 VAC / 4.5 A -> Stator bias; footprint TerminalBlock_Phoenix:TerminalBlock_Phoenix_MKDS-1,5-2-5.08_1x02_P5.08mm_Horizontal -> Connector_Molex:Molex_KK-396_A-41791-0002_1x02_P3.96mm_Vertical
- J6: value 10.5 VAC / 4.5 A -> HV-L; footprint TerminalBlock_Phoenix:TerminalBlock_Phoenix_MKDS-1,5-2-5.08_1x02_P5.08mm_Horizontal -> Connector_Molex:Molex_KK-396_A-41791-0004_1x04_P3.96mm_Vertical
- J7: value Stator bias -> HV-R; footprint Connector_Molex:Molex_KK-396_A-41791-0002_1x02_P3.96mm_Vertical -> Connector_Molex:Molex_KK-396_A-41791-0004_1x04_P3.96mm_Vertical
- J8: value HV-L -> HEATERS-LEFT; footprint Connector_Molex:Molex_KK-396_A-41791-0004_1x04_P3.96mm_Vertical -> Connector_Molex:Molex_KK-396_A-41791-0002_1x02_P3.96mm_Vertical
- J9: value HV-R -> HEATERS-RIGHT; footprint Connector_Molex:Molex_KK-396_A-41791-0004_1x04_P3.96mm_Vertical -> Connector_Molex:Molex_KK-396_A-41791-0002_1x02_P3.96mm_Vertical
- moved J6 265.7 mm to (194.8, 118.6)
- moved C3 140.5 mm to (230.6, 93.2), turned to -90 degrees
- moved C1 133.5 mm to (106.3, 103.5)
- moved C4 133.5 mm to (53.3, 109.2)
- moved CHASSIS1 133.5 mm to (34.9, 133.0)
- moved D1 133.5 mm to (73.9, 129.2)
- moved D10 133.5 mm to (268.6, 88.4)
- moved D13 133.5 mm to (109.0, 134.2)
- moved D14 133.5 mm to (100.5, 129.2)
- moved D16 133.5 mm to (172.4, 129.2)
- moved D18 133.5 mm to (185.9, 129.1)
- moved D20 133.5 mm to (234.0, 128.8)
- moved D22 133.5 mm to (220.5, 128.8)
- moved D3 133.5 mm to (60.4, 129.2)
- moved D8 133.5 mm to (263.8, 92.6)
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Connections:
- C7 pad 1: Net-(J10-Pin_1) -> Net-(J8-Pin_1)
- J5 pad 1: /COLEMAN_RAW_DC_LEFT/AC1 -> Net-(J5-Pin_1)
- J5 pad 2: /COLEMAN_RAW_DC_LEFT/AC2 -> Net-(J5-Pin_1)
- J6 pad 1: /COLEMAN_RAW_DC_RIGHT/AC1 -> /HV_STABI1/DC+
- J6 pad 2: /COLEMAN_RAW_DC_RIGHT/AC2 -> GND
- J7 pad 1: Net-(J7-Pin_1) -> /HV_STABI1/DC+
- J7 pad 2: Net-(J7-Pin_1) -> GND
- J8 pad 1: /HV_STABI1/DC+ -> Net-(J8-Pin_1)
- J9 pad 1: /HV_STABI1/DC+ -> Net-(J8-Pin_1)
- Q1 pad 1: Net-(J10-Pin_1) -> Net-(J8-Pin_1)
- R14 pad 1: Net-(J7-Pin_1) -> Net-(J5-Pin_1)
- R8 pad 1: Net-(J10-Pin_1) -> Net-(J8-Pin_1)
- R9 pad 2: Net-(J10-Pin_1) -> Net-(J8-Pin_1)
- RV1 pad 3: Net-(J10-Pin_1) -> Net-(J8-Pin_1)
- U1 pad 2: Net-(J10-Pin_1) -> Net-(J8-Pin_1)
- U2 pad 4: Net-(J10-Pin_1) -> Net-(J8-Pin_1)
- U2 pad 8: Net-(J10-Pin_1) -> Net-(J8-Pin_1)
Routing:
- net /HV_STABI3/DC-: track 0.00 -> 95.8 mm
- net /HV_STABI3/RSET: track 0.00 -> 46.6 mm
- net /HV_STABI3/CAP: track 0.00 -> 37.1 mm
- net Net-(Q11-S): track 0.00 -> 13.2 mm
- net Net-(Q13-S): track 0.00 -> 13.0 mm
- net Net-(R30-Pad2): track 0.00 -> 9.78 mm
- net Net-(Q11-G): track 0.00 -> 6.18 mm
- net Net-(Q12-G): track 0.00 -> 5.90 mm

Commit message: up
Parts:
- moved C6 15.0 mm to (254.5, 108.5), turned to 0 degrees
- moved C1 12.1 mm to (112.6, 93.2), turned to -90 degrees
- moved C2 11.3 mm to (171.6, 93.2), turned to -90 degrees
- moved Q2 7.17 mm to (263.7, 86.9)
- moved R11 6.27 mm to (270.5, 80.0)
- moved H3 5.75 mm to (253.1, 84.6)
- moved D10 3.84 mm to (269.7, 92.1), turned to -90 degrees
- moved D9 2.85 mm to (265.8, 99.7)
- moved D8 1.84 mm to (262.0, 92.1)
- moved J5 1.05 mm to (269.1, 131.0)
- moved D7 0.92 mm to (258.2, 92.1)
- moved C5 0.67 mm to (254.5, 118.5)
- moved C9 0.66 mm to (254.5, 72.5)
- moved D5 0.60 mm to (254.4, 99.7)
- moved H2 0.59 mm to (254.0, 133.2)
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Other:
- board text added: "OSDEHA mbrennwa@diyAudio"

Commit message: rearrange psu pcb
Parts:
- moved D21 222.5 mm to (80.6, -31.9), turned to -90 degrees
- moved D23 221.2 mm to (69.1, -31.9), turned to -90 degrees
- moved D20 218.2 mm to (86.4, -31.9)
- moved J3 218.1 mm to (99.2, -29.8)
- moved D22 216.9 mm to (74.9, -31.9)
- moved R28 214.8 mm to (105.2, -42.6)
- moved C3 214.5 mm to (86.7, -65.9)
- moved Q12 214.5 mm to (82.4, -81.8)
- moved Q13 214.5 mm to (80.8, -99.2)
- moved Q14 214.5 mm to (96.6, -98.2)
- moved R3 214.5 mm to (70.9, -89.7)
- moved R33 214.5 mm to (98.6, -82.5)
- moved RV4 214.5 mm to (76.2, -83.1)
- moved C14 214.5 mm to (57.4, -98.8)
- moved Q11 214.5 mm to (86.5, -84.3)
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Routing:
- net /HV_STABI3/CAP: track 37.1 -> 0.00 mm
- net /HV_STABI3/RSET: track 46.6 -> 12.4 mm
- net /HV_STABI3/DC-: track 95.8 -> 66.5 mm
- net Net-(Q11-S): track 13.2 -> 0.00 mm
- net Net-(Q13-S): track 13.0 -> 0.00 mm
- net Net-(R30-Pad2): track 9.78 -> 0.00 mm
- net Net-(Q11-G): track 6.18 -> 0.00 mm
- net Net-(Q12-G): track 5.90 -> 0.00 mm

Commit message: up
Parts:
- moved R19 229.4 mm to (228.2, -129.4)
- moved R20 229.4 mm to (224.0, -134.9)
- moved R21 229.4 mm to (233.5, -129.4)
- moved RV2 229.4 mm to (210.4, -121.2)
- moved R18 229.4 mm to (209.1, -136.7)
- moved Q3 229.4 mm to (224.3, -122.3)
- moved Q4 229.4 mm to (221.7, -126.4)
- moved Q5 229.4 mm to (215.8, -142.5)
- moved Q6 229.4 mm to (229.4, -134.3)
- moved R1 229.4 mm to (204.6, -136.8)
- moved R17 229.4 mm to (217.5, -119.3)
- moved Q10 221.8 mm to (157.6, -153.4)
- moved Q7 221.8 mm to (154.7, -141.0)
- moved Q8 221.8 mm to (152.1, -145.1)
- moved Q9 221.8 mm to (142.3, -161.0)
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Connections:
- J1 pad 1: /HV_STABI1/AC1 -> Net-(J1-Pin_1)
- J1 pad 2: Net-(J1-Pin_2) -> /HV_STABI1/AC1
- J2 pad 1: Net-(J2-Pin_1) -> /HV_STABI2/AC1
- J2 pad 2: /HV_STABI2/AC1 -> Net-(J2-Pin_2)
- K1 pad 11: /HV_STABI1/AC2 -> /HV_STABI2/AC2
- K1 pad 14: Net-(J1-Pin_2) -> Net-(J2-Pin_2)
- K1 pad 21: /HV_STABI2/AC2 -> /HV_STABI1/AC2
- K1 pad 24: Net-(J2-Pin_1) -> Net-(J1-Pin_1)
Routing:
- net /HV_STABI3/DC-: track 66.5 -> 0.00 mm
- net /HV_STABI3/RSET: track 12.4 -> 0.00 mm

Commit message: up
Parts:
- moved Q8 244.1 mm to (172.4, 98.2), turned to 90 degrees
- moved Q9 243.5 mm to (170.8, 80.8)
- moved R26 243.0 mm to (179.9, 87.5)
- moved R25 239.7 mm to (169.7, 91.6), turned to 0 degrees
- moved R23 238.5 mm to (183.7, 97.4)
- moved Q7 237.7 mm to (176.5, 95.6), turned to -90 degrees
- moved RV3 237.1 mm to (166.2, 96.9)
- moved Q10 236.9 mm to (186.6, 81.8)
- moved R27 236.5 mm to (188.5, 97.4)
- moved R2 235.9 mm to (160.8, 80.1)
- moved R24 235.9 mm to (165.2, 80.1)
- moved R21 231.2 mm to (188.5, 97.4), turned to 90 degrees
- moved Q4 229.9 mm to (172.4, 98.2), turned to 90 degrees
- moved Q5 227.8 mm to (170.8, 80.8)
- moved Q3 223.1 mm to (176.5, 95.6), turned to -90 degrees
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
Commit message: psu pcb
Parts:
- R11: footprint Resistor_THT:R_Axial_DIN0207_L6.3mm_D2.5mm_P10.16mm_Horizontal -> Resistor_THT:R_Axial_DIN0207_L6.3mm_D2.5mm_P2.54mm_Vertical
- moved R20 67.7 mm to (238.2, 87.6)
- moved R18 66.6 mm to (223.4, 80.2)
- moved R1 64.7 mm to (219.1, 80.2), turned to -90 degrees
- moved R19 60.8 mm to (228.0, 91.6)
- moved Q3 58.3 mm to (234.7, 95.7)
- moved Q5 58.3 mm to (229.0, 80.8)
- moved Q6 58.3 mm to (244.9, 81.8)
- moved R21 58.3 mm to (246.8, 97.5)
- moved RV2 58.3 mm to (224.4, 97.0)
- moved Q4 58.3 mm to (230.7, 98.2)
- moved R17 57.5 mm to (242.0, 97.5)
- moved R11 13.7 mm to (258.9, 103.7), turned to -90 degrees
- moved C10 3.00 mm to (255.9, 84.4)
- moved C9 3.00 mm to (255.9, 94.4)
- moved R12 3.00 mm to (251.7, 97.6)
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