File: kicad/powersupply/OSDEHA_PSU.kicad_pcb (KiCad board)
At the start: 2 copper layers, 104 parts, among them J1 340 VAC / 220 mA, J2 340 VAC / 220 mA, J3 420 VAC / 75 mA, J4 9 VAC / 4.5 A, J5 Stator bias, J6 HV-L, J7 HV-R, J8 HEATERS-LEFT, J9 HEATERS-RIGHT, K1 RT424006, Q1 BD138, Q10 BC550, Q11 LND150, Q12 LND150, Q13 NTHL1000N170M1, Q14 BC550, Q2 10M90S, Q3 LND150, Q4 LND150, Q5 NTHL1000N170M1, Q6 BC550, Q7 LND150, Q8 LND150, Q9 NTHL1000N170M1, U1 LM1085-ADJ, U2 NE555P

Commit message: psu pcb
Routing:
- net Earth_Protective: track 0.00 -> 84.3 mm
- net /HV_STABI1/AC2: track 0.00 -> 23.4 mm
- net /HV_STABI1/AC1: track 0.00 -> 18.4 mm
- net Net-(J1-Pin_1): track 0.00 -> 13.4 mm
- net Net-(J2-Pin_2): track 0.00 -> 13.3 mm
- added copper zone on F.Cu, net GND
Changed lines of the file:
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@@
     (effects (font (size 1.5 1.5) (thickness 0.3) bold) (justify left bottom))
+  )
+  (segment (start 225.027 150.672501) (end 239.644666 150.672501) (width 2) (layer "F.Cu") (net 9))
+  (segment (start 239.644666 150.672501) (end 242.224666 148.092501) (width 2) (layer "F.Cu") (net 9))
+  (segment (start 224.917 150.782501) (end 225.027 150.672501) (width 2) (layer "F.Cu") (net 9))
+  (segment (start 43.688 112.088) (end 44.45 112.85) (width 5) (layer "F.Cu") (net 15))
+  (segment (start 44.45 136.017) (end 38.735 141.732) (width 5) (layer "F.Cu") (net 15))
+  (segment (start 48.895 85.725) (end 43.688 90.932) (width 5) (layer "F.Cu") (net 15))
+  (segment (start 38.862 141.859) (end 38.735 141.732) (width 2) (layer "F.Cu") (net 15))
+  (segment (start 38.862 152.019) (end 38.862 141.859) (width 5) (layer "F.Cu") (net 15))
+  (segment (start 44.45 110.236) (end 44.45 112.85) (width 5) (layer "F.Cu") (net 15))
+  (segment (start 38.608 112.85) (end 44.45 112.85) (width 5) (layer "F.Cu") (net 15))
+  (segment (start 44.45 112.85) (end 44.45 136.017) (width 5) (layer "F.Cu") (net 15))
+  (segment (start 43.688 90.932) (end 43.688 112.088) (width 5) (layer "F.Cu") (net 15))
+  (segment (start 44.939 110.725) (end 44.45 110.236) (width 2) (layer "F.Cu") (net 15))
+  (segment (start 48.895 110.725) (end 44.939 110.725) (width 5) (layer "F.Cu") (net 15))
+  (segment (start 209.249 147.982501) (end 230.6 147.982501) (width 2) (layer "F.Cu") (net 28))
+  (segment (start 230.6 147.982501) (end 230.71 148.092501) (width 2) (layer "F.Cu") (net 28))
+  (segment (start 207.899 149.332501) (end 209.249 147.982501) (width 2) (layer "F.Cu") (net 28))
+  (segment (start 207.899 154.372501) (end 216.247 154.372501) (width 2) (layer "F.Cu") (net 62))
+  (segment (start 216.247 154.372501) (end 219.837 150.782501) (width 2) (layer "F.Cu") (net 62))
+  (segment (start 200.399 154.372501) (end 192.157 154.372501) (width 2) (layer "F.Cu") (net 63))
+  (segment (start 192.157 154.372501) (end 188.567 150.782501) (width 2) (layer "F.Cu") (net 63))
+  (zone (net 2) (net_name "GND") (layer "F.Cu") (hatch edge 0.5)
+    (connect_pads (clearance 0.5))
+    (min_thickness 0.25) (filled_areas_thickness no)
+    (fill (thermal_gap 0.5) (thermal_bridge_width 0.5))
+    (polygon
+      (pts
+        (xy 279.146 162.306)
+        (xy 278.892 69.342)
+        (xy 23.876 69.342)
+        (xy 24.384 162.814)
+        (xy 279.654 162.814)
+      )
+    )
   )
   (group "" (id 03a4125e-89cb-46b6-831d-42ff19693114)

Commit message: pcb psu
Parts:
- moved D10 7.62 mm to (271.0, 118.6), turned to 90 degrees
- moved D8 7.62 mm to (263.4, 118.6), turned to 90 degrees
- moved D9 7.62 mm to (267.2, 111.0), turned to -90 degrees
- moved H3 3.00 mm to (249.2, 105.2)
Routing:
- net /HV_STABI1/DC+: track 0.00 -> 149.5 mm
- net Net-(D8-K): track 0.00 -> 87.5 mm
- net /HV_STABI1/CAP: track 0.00 -> 54.2 mm
- net /HV_STABI1/AC1: track 18.4 -> 55.7 mm
- net Net-(D7-K): track 0.00 -> 32.2 mm
- net Net-(D5-K): track 0.00 -> 21.0 mm
- net Net-(Q5-S): track 0.00 -> 14.0 mm
- net /HV_STABI3/DC-: track 0.00 -> 11.8 mm
- net /HV_STABI2/DC-: track 0.00 -> 11.8 mm
- net Net-(J5-Pin_1): track 0.00 -> 11.0 mm
- net /HV_STABI1/RSET: track 0.00 -> 6.59 mm
- net Net-(Q2-G): track 0.00 -> 5.30 mm
- net Net-(C9-Pad1): track 0.00 -> 4.46 mm
- net Net-(C10-Pad1): track 0.00 -> 4.45 mm
- net Net-(D8-A): track 0.00 -> 3.82 mm
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
Commit message: psu pcb
Parts:
- R5, R6: footprint Resistor_THT:R_Axial_DIN0207_L6.3mm_D2.5mm_P10.16mm_Horizontal -> Resistor_THT:R_Axial_DIN0207_L6.3mm_D2.5mm_P2.54mm_Vertical
- moved R5 103.3 mm to (249.4, 102.1)
- moved R6 101.4 mm to (249.4, 105.6)
- moved H3 30.6 mm to (218.6, 104.6)
Routing:
- net /HV_STABI1/RSET: track 6.59 -> 73.0 mm
- net /HV_STABI1/CAP: track 54.2 -> 99.2 mm
- net Net-(Q3-S): track 0.00 -> 17.7 mm
- net Net-(D5-A): track 0.00 -> 12.1 mm
- net Net-(R18-Pad2): track 0.00 -> 9.78 mm
- net Net-(Q5-G): track 0.00 -> 7.16 mm
- net Net-(D6-K): track 0.00 -> 5.99 mm
- net Net-(Q3-G): track 0.00 -> 5.80 mm
- net Net-(Q4-G): track 0.00 -> 5.76 mm
- net /HV_STABI1/DC+: track 149.5 -> 154.7 mm
- net Net-(Q3-D): track 0.00 -> 4.06 mm

Commit message: pcb psu
Parts:
- moved C14 37.5 mm to (85.3, 118.7), turned to 90 degrees
- moved R3 10.2 mm to (100.3, 80.0), turned to -90 degrees
- moved R16 5.61 mm to (251.8, 132.5), turned to 90 degrees
- moved R22 5.61 mm to (192.5, 132.5), turned to 90 degrees
- moved R28 5.61 mm to (133.1, 132.5), turned to 90 degrees
Connections:
- J3 pad 1: /HV_STABI3/AC1 -> /HV_STABI3/AC2
- J3 pad 2: /HV_STABI3/AC2 -> /HV_STABI3/AC1
- J4 pad 1: Net-(D1-K) -> Net-(D2-A)
- J4 pad 2: Net-(D2-A) -> Net-(D1-K)
Routing:
- net /HV_STABI2/DC-: track 11.8 -> 185.7 mm
- net Net-(D6-K): track 5.99 -> 163.4 mm, vias 0 -> 2
- net /HV_STABI3/DC-: track 11.8 -> 155.9 mm
- net Net-(J8-Pin_1): track 0.00 -> 112.8 mm
- net /HV_STABI3/CAP: track 0.00 -> 107.4 mm
- net /HV_STABI2/CAP: track 0.00 -> 107.2 mm
- net Net-(D3-K): track 0.00 -> 98.1 mm
- net /HV_STABI3/RSET: track 0.00 -> 73.2 mm
- net /HV_STABI2/RSET: track 0.00 -> 73.1 mm
- net Net-(U2-THR): track 0.00 -> 61.6 mm
- net /HV_STABI2/AC2: track 0.00 -> 54.4 mm
- net /HV_STABI3/AC2: track 0.00 -> 42.9 mm
- net Net-(D2-A): track 0.00 -> 28.2 mm
- net Net-(D1-K): track 0.00 -> 27.6 mm
- net Net-(U2-Q): track 0.00 -> 20.2 mm
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
Commit message: pcb psu
Routing:
- net Earth_Protective: track 84.3 -> 84.9 mm
Changed lines of the file:
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@@
   (segment (start 252.309 84.407) (end 251.674 85.042) (width 2) (layer "B.Cu") (net 14))
   (segment (start 255.858 84.407) (end 252.309 84.407) (width 2) (layer "B.Cu") (net 14))
+  (segment (start 44.958 113.358) (end 44.958 135.509) (width 7) (layer "F.Cu") (net 15))
   (segment (start 43.688 112.088) (end 44.45 112.85) (width 5) (layer "F.Cu") (net 15))
-  (segment (start 44.45 136.017) (end 38.735 141.732) (width 5) (layer "F.Cu") (net 15))
-  (segment (start 48.895 85.725) (end 43.688 90.932) (width 5) (layer "F.Cu") (net 15))
+  (segment (start 44.45 112.85) (end 44.958 113.358) (width 7) (layer "F.Cu") (net 15))
+  (segment (start 43.4848 93.2688) (end 43.4848 111.8848) (width 7) (layer "F.Cu") (net 15))
+  (segment (start 48.895 85.725) (end 48.895 87.8586) (width 7) (layer "F.Cu") (net 15))
   (segment (start 38.862 141.859) (end 38.735 141.732) (width 2) (layer "F.Cu") (net 15))
-  (segment (start 38.862 152.019) (end 38.862 141.859) (width 5) (layer "F.Cu") (net 15))
+  (segment (start 38.862 152.019) (end 38.862 141.859) (width 7) (layer "F.Cu") (net 15))
+  (segment (start 44.958 135.509) (end 38.735 141.732) (width 7) (layer "F.Cu") (net 15))
   (segment (start 44.45 110.236) (end 44.45 112.85) (width 5) (layer "F.Cu") (net 15))
+  (segment (start 43.4848 111.8848) (end 43.688 112.088) (width 7) (layer "F.Cu") (net 15))
   (segment (start 38.608 112.85) (end 44.45 112.85) (width 5) (layer "F.Cu") (net 15))
-  (segment (start 44.45 112.85) (end 44.45 136.017) (width 5) (layer "F.Cu") (net 15))
-  (segment (start 43.688 90.932) (end 43.688 112.088) (width 5) (layer "F.Cu") (net 15))
+  (segment (start 48.895 87.8586) (end 43.4848 93.2688) (width 7) (layer "F.Cu") (net 15))
   (segment (start 44.939 110.725) (end 44.45 110.236) (width 2) (layer "F.Cu") (net 15))
   (segment (start 48.895 110.725) (end 44.939 110.725) (width 5) (layer "F.Cu") (net 15))

Commit message: psu pcb
Parts:
- moved R4 17.0 mm to (57.3, 144.5)
- moved H1 0.83 mm to (38.7, 81.7)
Routing:
- net Net-(D3-K): track 98.1 -> 86.9 mm
- net Net-(Q12-G): track 0.00 -> 5.76 mm
- net Net-(Q8-G): track 0.00 -> 5.76 mm
Other:
- board outline added: 239.3 x 78.3 mm

Commit message: PSU PCB
Parts:
- removed H1, H2, H3: MountingHole, MountingHole:MountingHole_3.2mm_M3
- added REF**: MountingHole_3.2mm_M3, MountingHole:MountingHole_3.2mm_M3, F.Cu at (37.4, 81.3)
- added REF**: MountingHole_3.2mm_M3, MountingHole:MountingHole_3.2mm_M3, F.Cu at (255.6, 152.7)
- added REF**: MountingHole_3.2mm_M3, MountingHole:MountingHole_3.2mm_M3, F.Cu at (218.9, 104.3)
- moved C7 2.50 mm to (90.2, 124.2), turned to -90 degrees
- moved C8 2.50 mm to (81.2, 124.2), turned to -90 degrees
- moved CHASSIS1 1.60 mm to (37.4, 152.7)
Routing:
- net Net-(J8-Pin_1): track 112.8 -> 116.9 mm
- net Net-(U2-THR): track 61.6 -> 57.7 mm
- net Earth_Protective: track 85.0 -> 86.2 mm
- net /HV_STABI2/DC-: track 185.7 -> 186.6 mm
- net /HV_STABI1/AC1: track 55.7 -> 56.2 mm

Commit message: PSU PCB
Parts:
- moved Q5 0.08 mm to (229.0, 80.8)
Routing:
- net /HV_STABI2/RSET: track 73.1 -> 74.0 mm
- net /HV_STABI1/RSET: track 73.0 -> 73.9 mm
- net /HV_STABI3/RSET: track 73.2 -> 74.1 mm
Changed lines of the file:
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@@
   )
   (footprint "Package_TO_SOT_THT:TO-247-3_Vertical" (layer "F.Cu")
-    (at 229.0334 80.8482)
+    (at 229.0334 80.772)
     (descr "TO-247-3, Vertical, RM 5.45mm, see https://toshiba.semicon-storage.com/us/product/mosfet/to-247-4l.html")
     (tags "TO-247-3 Vertical RM 5.45mm")
@@
   (segment (start 48.895 110.725) (end 44.939 110.725) (width 5) (layer "F.Cu") (net 15))
   (segment (start 182.448 87.503) (end 182.702 87.249) (width 2) (layer "F.Cu") (net 16))
+  (segment (start 178.8666 87.5284) (end 173.9392 87.5284) (width 2) (layer "F.Cu") (net 16))
   (segment (start 182.7276 84.444) (end 185.3936 81.778) (width 1) (layer "F.Cu") (net 16))
-  (segment (start 176.592 85.203) (end 164.936 85.203) (width 2) (layer "F.Cu") (net 16))
   (segment (start 164.16 84.9376) (end 164.16 85.979) (width 2) (layer "F.Cu") (net 16))
   (segment (start 164.16 80.137) (end 164.16 84.9376) (width 2) (layer "F.Cu") (net 16))
+  (segment (start 173.9392 87.5284) (end 171.3484 84.9376) (width 2) (layer "F.Cu") (net 16))
   (segment (start 182.7276 87.26) (end 182.7276 84.444) (width 1) (layer "F.Cu") (net 16))
   (segment (start 144.78 118.699) (end 144.78 105.359) (width 2) (layer "F.Cu") (net 16))
+  (segment (start 178.892 87.503) (end 178.8666 87.5284) (width 2) (layer "F.Cu") (net 16))
   (segment (start 144.78 105.359) (end 159.842 90.297) (width 2) (layer "F.Cu") (net 16))
   (segment (start 178.892 87.503) (end 182.448 87.503) (width 2) (layer "F.Cu") (net 16))
-  (segment (start 178.892 87.503) (end 176.592 85.203) (width 2) (layer "F.Cu") (net 16))
+  (segment (start 171.3484 84.9376) (end 164.16 84.9376) (width 2) (layer "F.Cu") (net 16))
   (segment (start 164.936 85.203) (end 164.16 85.979) (width 2) (layer "F.Cu") (net 16))
   (segment (start 164.16 85.979) (end 159.842 90.297) (width 2) (layer "F.Cu") (net 16))
   (segment (start 241.7224 87.5792) (end 238.1664 87.5792) (width 2) (layer "F.Cu") (net 17))
   (segment (start 204.089 118.699) (end 204.089 105.4006) (width 2) (layer "F.Cu") (net 17))
+  (segment (start 233.1975 87.5792) (end 230.6067 84.9884) (width 2) (layer "F.Cu") (net 17))
   (segment (start 241.9764 87.3252) (end 241.9764 84.5092) (width 1) (layer "F.Cu") (net 17))
   (segment (start 204.089 105.4006) (end 219.1164 90.3732) (width 2) (layer "F.Cu") (net 17))
-  (segment (start 238.1664 87.5792) (end 235.8664 85.2792) (width 2) (layer "F.Cu") (net 17))
+  (segment (start 238.1249 87.5792) (end 233.1975 87.5792) (width 2) (layer "F.Cu") (net 17))
   (segment (start 223.4344 86.0552) (end 219.1164 90.3732) (width 2) (layer "F.Cu") (net 17))
-  (segment (start 235.8664 85.2792) (end 224.2104 85.2792) (width 2) (layer "F.Cu") (net 17))
+  (segment (start 230.6067 84.9884) (end 223.4183 84.9884) (width 2) (layer "F.Cu") (net 17))
   (segment (start 241.9764 84.5092) (end 244.6424 81.8432) (width 1) (layer "F.Cu") (net 17))
   (segment (start 241.9764 87.3252) (end 241.7224 87.5792) (width 2) (layer "F.Cu") (net 17))
@@
   (segment (start 223.4344 80.2132) (end 223.4344 86.0552) (width 2) (layer "F.Cu") (net 17))
   (segment (start 85.344 105.172) (end 100.346 90.17) (width 2) (layer "F.Cu") (net 18))
-  (segment (start 119.396 87.376) (end 117.096 85.076) (width 2) (layer "F.Cu") (net 18))
   (segment (start 105.44 85.076) (end 104.664 85.852) (width 2) (layer "F.Cu") (net 18))
+  (segment (start 114.4271 87.376) (end 111.8363 84.7852) (width 2) (layer "F.Cu") (net 18))
   (segment (start 122.952 87.376) (end 123.206 87.122) (width 2) (layer "F.Cu") (net 18))
+  (segment (start 119.3545 87.376) (end 114.4271 87.376) (width 2) (layer "F.Cu") (net 18))
+  (segment (start 111.8363 84.7852) (end 104.6479 84.7852) (width 2) (layer "F.Cu") (net 18))
   (segment (start 123.2408 84.2916) (end 125.9068 81.6256) (width 1) (layer "F.Cu") (net 18))
   (segment (start 123.2408 87.1076) (end 123.2408 84.2916) (width 1) (layer "F.Cu") (net 18))
   (segment (start 85.344 118.699) (end 85.344 105.172) (width 2) (layer "F.Cu") (net 18))
-  (segment (start 117.096 85.076) (end 105.44 85.076) (width 2) (layer "F.Cu") (net 18))
   (segment (start 104.664 85.852) (end 100.346 90.17) (width 2) (layer "F.Cu") (net 18))
   (segment (start 119.396 87.376) (end 122.952 87.376) (width 2) (layer "F.Cu") (net 18))
