File: kicad/powersupply_DHTfilaments/COLEMAN_RAW_DC.kicad_sch (KiCad schematic)
At the start: 9 parts

Commit message: up
Parts:
- R1: footprint Resistor_THT:R_Axial_DIN0207_L6.3mm_D2.5mm_P10.16mm_Horizontal -> Resistor_THT:R_Axial_DIN0207_L6.3mm_D2.5mm_P2.54mm_Vertical
- R2, R3: footprint Resistor_THT:R_Axial_DIN0614_L14.3mm_D5.7mm_P15.24mm_Horizontal -> Resistor_THT:R_Axial_DIN0614_L14.3mm_D5.7mm_P5.08mm_Vertical
Changed lines of the file:
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@@
 		)
 		(instances
-			(project "OSDEHA_powersupply_colemanreg"
+			(project "OSDEHA_powersupply_DHTfil"
 				(path "/6a766a35-7f7e-4680-bf64-1ed131aec470/5c8de33b-0aec-4bd3-8a06-d4311bc9100c"
 					(reference "D4")
@@
 		)
 		(instances
-			(project "OSDEHA_powersupply_colemanreg"
+			(project "OSDEHA_powersupply_DHTfil"
 				(path "/6a766a35-7f7e-4680-bf64-1ed131aec470/5c8de33b-0aec-4bd3-8a06-d4311bc9100c"
 					(reference "D2")
@@
 			)
 		)
-		(property "Footprint" "Resistor_THT:R_Axial_DIN0614_L14.3mm_D5.7mm_P15.24mm_Horizontal"
+		(property "Footprint" "Resistor_THT:R_Axial_DIN0614_L14.3mm_D5.7mm_P5.08mm_Vertical"
 			(at 130.81 89.408 90)
 			(effects
@@
 		)
 		(instances
-			(project "OSDEHA_powersupply_colemanreg"
+			(project "OSDEHA_powersupply_DHTfil"
 				(path "/6a766a35-7f7e-4680-bf64-1ed131aec470/5c8de33b-0aec-4bd3-8a06-d4311bc9100c"
 					(reference "R3")
@@
 		)
 		(instances
-			(project "OSDEHA_powersupply_colemanreg"
+			(project "OSDEHA_powersupply_DHTfil"
 				(path "/6a766a35-7f7e-4680-bf64-1ed131aec470/5c8de33b-0aec-4bd3-8a06-d4311bc9100c"
 					(reference "D3")
@@
 		)
 		(instances
-			(project "OSDEHA_powersupply_colemanreg"
+			(project "OSDEHA_powersupply_DHTfil"
 				(path "/6a766a35-7f7e-4680-bf64-1ed131aec470/5c8de33b-0aec-4bd3-8a06-d4311bc9100c"
 					(reference "D1")
@@
 		)
 		(instances
-			(project "OSDEHA_powersupply_colemanreg"
+			(project "OSDEHA_powersupply_DHTfil"
 				(path "/6a766a35-7f7e-4680-bf64-1ed131aec470/5c8de33b-0aec-4bd3-8a06-d4311bc9100c"
 					(reference "C1")
@@
 		)
 		(instances
-			(project "OSDEHA_powersupply_colemanreg"
+			(project "OSDEHA_powersupply_DHTfil"
 				(path "/6a766a35-7f7e-4680-bf64-1ed131aec470/5c8de33b-0aec-4bd3-8a06-d4311bc9100c"
 					(reference "C2")
@@
 			)
 		)
-		(property "Footprint" "Resistor_THT:R_Axial_DIN0207_L6.3mm_D2.5mm_P10.16mm_Horizontal"
+		(property "Footprint" "Resistor_THT:R_Axial_DIN0207_L6.3mm_D2.5mm_P2.54mm_Vertical"
 			(at 104.902 74.93 90)
 			(effects
@@
 		)
 		(instances
-			(project "OSDEHA_powersupply_colemanreg"
+			(project "OSDEHA_powersupply_DHTfil"
 				(path "/6a766a35-7f7e-4680-bf64-1ed131aec470/5c8de33b-0aec-4bd3-8a06-d4311bc9100c"
 					(reference "R1")
@@
 			)
 		)
-		(property "Footprint" "Resistor_THT:R_Axial_DIN0614_L14.3mm_D5.7mm_P15.24mm_Horizontal"
+		(property "Footprint" "Resistor_THT:R_Axial_DIN0614_L14.3mm_D5.7mm_P5.08mm_Vertical"
 			(at 130.81 64.008 90)
 			(effects
@@
 		)
 		(instances
-			(project "OSDEHA_powersupply_colemanreg"
+			(project "OSDEHA_powersupply_DHTfil"
 				(path "/6a766a35-7f7e-4680-bf64-1ed131aec470/5c8de33b-0aec-4bd3-8a06-d4311bc9100c"
 					(reference "R2")
