File: kicad/powersupply_DHTfilaments/OSDEHA_powersupply_DHTfil.kicad_pcb (KiCad board)
At the start: 2 copper layers, 98.5 x 26 mm, 15 parts

Commit message: add version label to DC raw supply (schematic and PCB)
Other:
- board text added: "mbrennwa.github.io/OSDEHA V20240515"
- board text removed: "mbrennwa.github.io/OSDEHA"
Changed lines of the file:
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@@
 		(layer "Edge.Cuts")
 	)
-	(gr_text "mbrennwa.github.io/OSDEHA"
+	(gr_text "mbrennwa.github.io/OSDEHA\nV20240515"
 		(at 158.25 93.65 0)
 		(layer "B.SilkS")
