File: kicad/powersupply_new_layout/OSDEHA_PSU.kicad_pcb (KiCad board)
At the start: 2 copper layers, 239.3 x 78.3 mm, 114 parts, among them J1 340 VAC / 220 mA, J2 340 VAC / 220 mA, J3 420 VAC / 75 mA, J4 9 VAC / 4.5 A, J5 Stator bias, J6 HV-L, J7 HV-R, J8 HEATERS-LEFT, J9 HEATERS-RIGHT, K1 RT424006, Q1 BD138, Q10 BC550, Q11 LND150, Q12 LND150, Q13 NTHL1000N170M1, Q14 BC550, Q2 10M90S, Q3 LND150, Q4 LND150, Q5 NTHL1000N170M1, Q6 BC550, Q7 LND150, Q8 LND150, Q9 NTHL1000N170M1, U1 LM1085-ADJ, U2 NE555P

Commit message: up
Parts:
- added D24: 10 V, Diode_THT:D_DO-41_SOD81_P7.62mm_Horizontal, F.Cu at (171.4, 86.0)
- added D27: 1N4007, Diode_THT:D_DO-41_SOD81_P2.54mm_Vertical_KathodeUp, F.Cu at (182.2, 101.0)
- added Q3: LND150, Package_TO_SOT_THT:TO-92_HandSolder, F.Cu at (168.5, 92.2)
- added Q4: LND150, Package_TO_SOT_THT:TO-92_HandSolder, F.Cu at (168.5, 98.7)
- added Q5: NTHL1000N170M1, Package_TO_SOT_THT:TO-247-3_Vertical, F.Cu at (169.8, 80.8)
- added Q6: BC550, Package_TO_SOT_THT:TO-92_HandSolder, F.Cu at (186.5, 92.7)
- added R1: 866k, Resistor_THT:R_Axial_DIN0207_L6.3mm_D2.5mm_P10.16mm_Horizontal, F.Cu at (157.8, 79.0)
- added R17: 1k, Resistor_THT:R_Axial_DIN0207_L6.3mm_D2.5mm_P10.16mm_Horizontal, F.Cu at (161.2, 79.0)
- added R18: 1k, Resistor_THT:R_Axial_DIN0207_L6.3mm_D2.5mm_P10.16mm_Horizontal, F.Cu at (157.8, 91.9)
- added R19: 1k, Resistor_THT:R_Axial_DIN0207_L6.3mm_D2.5mm_P10.16mm_Horizontal, F.Cu at (174.2, 101.6)
- added R20: 300, Resistor_THT:R_Axial_DIN0207_L6.3mm_D2.5mm_P10.16mm_Horizontal, F.Cu at (164.8, 79.0)
- added R21: 2, Resistor_THT:R_Axial_DIN0207_L6.3mm_D2.5mm_P10.16mm_Horizontal, F.Cu at (185.8, 89.2)
- added R34: 1k, Resistor_THT:R_Axial_DIN0207_L6.3mm_D2.5mm_P10.16mm_Horizontal, F.Cu at (189.2, 89.2)
- added RV2: 1k, Potentiometer_THT:Potentiometer_Bourns_3296W_Vertical, F.Cu at (162.8, 94.4)
- moved R25 74.2 mm to (174.2, 101.6), turned to 90 degrees
- moved Q8 70.2 mm to (168.5, 98.7), turned to -90 degrees
- moved Q7 69.8 mm to (168.5, 92.2), turned to -90 degrees
- moved R23 68.2 mm to (161.2, 89.2), turned to 90 degrees
- moved R24 66.9 mm to (157.8, 91.9), turned to -90 degrees
- moved Q10 59.7 mm to (186.5, 92.7), turned to -90 degrees
- moved R27 58.6 mm to (185.8, 89.2), turned to 90 degrees
- moved R35 56.9 mm to (189.2, 89.2), turned to 90 degrees
- moved R26 56.4 mm to (164.8, 89.2), turned to 90 degrees
- moved RV3 56.2 mm to (162.8, 94.5), turned to 90 degrees
- moved R3 49.2 mm to (112.0, 71.1), turned to 90 degrees
- moved D25 42.5 mm to (171.4, 86.0)
- moved R2 27.5 mm to (157.8, 79.0), turned to -90 degrees
Routing:
- net /B-: track 111.4 -> 113.3 mm

Commit message: PCB layout work
Parts:
- removed the D24 at (171.4, 86.0)
- removed the D27 at (182.2, 101.0)
- removed the Q3 at (168.5, 92.2)
- removed the Q4 at (168.5, 98.7)
- removed the Q5 at (169.8, 80.8)
- removed the Q6 at (186.5, 92.7)
- removed the R1 at (157.8, 79.0)
- removed the R17 at (161.2, 79.0)
- removed the R18 at (157.8, 91.9)
- removed the R19 at (174.2, 101.6)
- removed the R20 at (164.8, 79.0)
- removed the R21 at (185.8, 89.2)
- removed the R34 at (189.2, 89.2)
- removed the RV2 at (162.8, 94.4)
- moved Q12 79.1 mm to (109.0, 98.6), turned to -90 degrees
- moved Q11 78.8 mm to (109.0, 92.1), turned to -90 degrees
- moved R30 74.9 mm to (98.2, 91.8), turned to -90 degrees
- moved R31 74.5 mm to (114.7, 101.5), turned to 90 degrees
- moved RV4 72.6 mm to (103.2, 94.3), turned to 90 degrees
- moved R29 65.4 mm to (101.7, 78.9), turned to -90 degrees
- moved Q14 60.9 mm to (127.0, 92.6), turned to -90 degrees
- moved R32 53.1 mm to (105.2, 78.9), turned to -90 degrees
- moved R33 52.2 mm to (126.2, 89.0), turned to 90 degrees
- moved R36 47.9 mm to (129.7, 89.0), turned to 90 degrees
- moved D26 45.4 mm to (111.9, 85.9)
- moved R3 15.8 mm to (98.2, 78.9), turned to -90 degrees
- moved R23 10.2 mm to (161.2, 79.0), turned to -90 degrees
- moved R26 10.2 mm to (164.7, 79.0), turned to -90 degrees
- moved C4 7.09 mm to (62.3, 123.3), turned to -90 degrees
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Routing:
- net /B2-: track 87.1 -> 158.4 mm
- net /B-: track 113.3 -> 184.5 mm
- net /HV_STABI3/CAP: track 62.6 -> 118.5 mm
- net /HV_STABI2/CAP: track 62.6 -> 118.3 mm
- net /HV_STABI3/RSET: track 0.00 -> 42.0 mm
- net /HV_STABI2/RSET: track 0.00 -> 41.9 mm
- net Net-(D25-K): track 0.00 -> 29.5 mm
- net Net-(D26-K): track 0.00 -> 29.5 mm
- net Net-(Q7-G): track 0.00 -> 18.1 mm
- net Net-(Q11-G): track 0.00 -> 18.1 mm
- net Net-(D6-K): track 162.8 -> 178.8 mm, vias 0 -> 4
- net Net-(D26-A): track 0.00 -> 15.6 mm
- net Net-(D25-A): track 0.00 -> 15.4 mm
- net Net-(Q7-S): track 0.00 -> 12.7 mm
- net Net-(Q11-S): track 0.00 -> 12.7 mm
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Other:
- board text added: "340 VAC"
- board text added: "420 VAC"
- board text added: "9 VAC"
- board text added: "BIAS"
- board text added: "HEATERS"
- board text added: "HIGH VOLTAGE"
- board text added: "mbrennwa.github.io/OSDEHA"
- board text removed: "OSDEHA mbrennwa@diyAudio"
