File: kicad/system_overview_boards/system_boards_overview.kicad_sch (KiCad schematic)
At the start: 0 parts

Commit message: up
Other:
- sheet Coleman Fil-Reg PCB (L1)1 renamed Coleman Fil-Reg PCB (R1)
- sheet Coleman Fil-Reg PCB (L2)1 renamed Coleman Fil-Reg PCB (R2)
Changed lines of the file:
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@@
 	(paper "A4")
 	(junction
-		(at 139.7 124.46)
+		(at 175.26 80.01)
 		(diameter 0)
 		(color 0 0 0 0)
 	)
 	(junction
-		(at 185.42 57.15)
+		(at 175.26 133.35)
 		(diameter 0)
 		(color 0 0 0 0)
 	)
 	(junction
-		(at 190.5 80.01)
+		(at 139.7 124.46)
+		(diameter 0)
+		(color 0 0 0 0)
+	)
+	(junction
+		(at 185.42 57.15)
 		(diameter 0)
 		(color 0 0 0 0)
@@
 	)
 	(junction
+		(at 180.34 52.07)
+		(diameter 0)
+		(color 0 0 0 0)
+	)
+	(junction
 		(at 85.09 63.5)
 		(diameter 0)
@@
 	(wire
 		(pts
+			(xy 180.34 147.32) (xy 180.34 52.07)
+		)
+		(stroke
+			(width 0)
+			(type default)
+		)
+	)
+	(wire
+		(pts
 			(xy 242.57 104.14) (xy 229.87 104.14)
 		)
@@
 	(wire
 		(pts
+			(xy 199.39 139.7) (xy 177.8 139.7)
+		)
+		(stroke
+			(width 0)
+			(type default)
+		)
+	)
+	(wire
+		(pts
 			(xy 186.69 54.61) (xy 199.39 54.61)
 		)
@@
 	(wire
 		(pts
+			(xy 175.26 133.35) (xy 175.26 127)
+		)
+		(stroke
+			(width 0)
+			(type default)
+		)
+	)
+	(wire
+		(pts
 			(xy 184.15 59.69) (xy 199.39 59.69)
 		)
@@
 	(wire
 		(pts
-			(xy 172.72 86.36) (xy 190.5 86.36)
+			(xy 172.72 86.36) (xy 175.26 86.36)
 		)
 		(stroke
@@
 	(wire
 		(pts
-			(xy 234.95 96.52) (xy 234.95 106.68)
+			(xy 175.26 144.78) (xy 199.39 144.78)
 		)
 		(stroke
@@
 	(wire
 		(pts
-			(xy 139.7 83.82) (xy 146.05 83.82)
+			(xy 234.95 96.52) (xy 234.95 106.68)
 		)
 		(stroke
@@
 	(wire
 		(pts
-			(xy 233.68 129.54) (xy 238.76 129.54)
+			(xy 139.7 83.82) (xy 146.05 83.82)
 		)
 		(stroke
@@
 	(wire
 		(pts
-			(xy 199.39 142.24) (xy 182.88 142.24)
+			(xy 233.68 129.54) (xy 238.76 129.54)
 		)
 		(stroke
@@
 	(wire
 		(pts
+			(xy 176.53 142.24) (xy 199.39 142.24)
+		)
+		(stroke
+			(width 0)
+			(type default)
+		)
+	)
+	(wire
+		(pts
 			(xy 233.68 72.39) (xy 242.57 72.39)
 		)
@@
 	(wire
 		(pts
+			(xy 176.53 130.81) (xy 172.72 130.81)
+		)
+		(stroke
+			(width 0)
+			(type default)
+		)
+	)
+	(wire
+		(pts
 			(xy 234.95 49.53) (xy 233.68 49.53)
 		)
@@
 	(wire
 		(pts
+			(xy 175.26 144.78) (xy 175.26 133.35)
+		)
+		(stroke
+			(width 0)
+			(type default)
+		)
+	)
+	(wire
+		(pts
+			(xy 175.26 80.01) (xy 190.5 80.01)
+		)
+		(stroke
+			(width 0)
+			(type default)
+		)
+	)
+	(wire
+		(pts
 			(xy 232.41 101.6) (xy 232.41 99.06)
 		)
@@
 	(wire
 		(pts
+			(xy 172.72 133.35) (xy 175.26 133.35)
+		)
+		(stroke
+			(width 0)
+			(type default)
+		)
+	)
+	(wire
+		(pts
 			(xy 190.5 44.45) (xy 220.98 44.45)
 		)
@@
 	(wire
 		(pts
-			(xy 190.5 80.01) (xy 190.5 86.36)
+			(xy 218.44 146.05) (xy 218.44 147.32)
+		)
+		(stroke
+			(width 0)
+			(type default)
+		)
+	)
+	(wire
+		(pts
+			(xy 175.26 80.01) (xy 175.26 86.36)
 		)
 		(stroke
@@
 	(wire
 		(pts
+			(xy 175.26 127) (xy 172.72 127)
+		)
+		(stroke
+			(width 0)
+			(type default)
+		)
+	)
+	(wire
+		(pts
+			(xy 177.8 139.7) (xy 177.8 124.46)
+		)
+		(stroke
+			(width 0)
+			(type default)
+		)
+	)
+	(wire
+		(pts
 			(xy 129.54 83.82) (xy 129.54 118.11)
 		)
@@
 	(wire
 		(pts
+			(xy 180.34 52.07) (xy 190.5 52.07)
+		)
+		(stroke
+			(width 0)
+			(type default)
+		)
+	)
+	(wire
+		(pts
 			(xy 236.22 49.53) (xy 265.43 49.53)
 		)
@@
 	(wire
 		(pts
+			(xy 176.53 142.24) (xy 176.53 130.81)
+		)
+		(stroke
+			(width 0)
+			(type default)
+		)
+	)
+	(wire
+		(pts
 			(xy 121.92 88.9) (xy 101.6 88.9)
 		)
@@
 	(wire
 		(pts
-			(xy 233.68 64.77) (xy 242.57 64.77)
+			(xy 218.44 147.32) (xy 180.34 147.32)
 		)
 		(stroke
@@
 	(wire
 		(pts
-			(xy 181.61 144.78) (xy 199.39 144.78)
+			(xy 233.68 64.77) (xy 242.57 64.77)
 		)
 		(stroke
@@
 	(wire
 		(pts
-			(xy 119.38 52.07) (xy 190.5 52.07)
+			(xy 119.38 52.07) (xy 180.34 52.07)
 		)
 		(stroke
@@
 	(wire
 		(pts
+			(xy 177.8 124.46) (xy 172.72 124.46)
+		)
+		(stroke
+			(width 0)
+			(type default)
+		)
+	)
+	(wire
+		(pts
 			(xy 193.04 124.46) (xy 199.39 124.46)
 		)
@@
 	(wire
 		(pts
-			(xy 172.72 80.01) (xy 190.5 80.01)
+			(xy 172.72 80.01) (xy 175.26 80.01)
 		)
 		(stroke
@@
 			(color 0 0 0 0.0000)
 		)
-		(property "Sheetname" "Coleman Fil-Reg PCB (L1)1"
+		(property "Sheetname" "Coleman Fil-Reg PCB (R1)"
 			(at 146.05 122.4784 0)
 			(effects
@@
 		)
 		(property "Sheetname" "Stax Socket"
-			(at 269.24 106.426 0)
+			(at 268.732 106.68 0)
 			(effects
 				(font
@@
 			(color 0 0 0 0.0000)
 		)
-		(property "Sheetname" "Coleman Fil-Reg PCB (L2)1"
+		(property "Sheetname" "Coleman Fil-Reg PCB (R2)"
 			(at 146.05 136.906 0)
 			(effects
@@
 		)
 		(property "Sheetname" "Mains Transformer (HTR+FIL)"
-			(at 38.1 110.998 0)
+			(at 37.846 130.048 0)
 			(effects
 				(font
