File: kicad/system_overview_boards/PSU_main.kicad_sch (KiCad schematic)
At the start: 0 parts

Commit message: system overview
Changed lines of the file:
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@@
 	(generator_version "8.0")
 	(paper "A4")
-	(hierarchical_label "HEATER- (R)"
-		(shape passive)
-		(at 142.24 62.23 0)
-		(fields_autoplaced yes)
-		(effects
-			(font
-				(size 1.27 1.27)
-			)
-			(justify left)
-		)
-	)
-	(hierarchical_label "HEATER+ (L)"
+	(hierarchical_label "HEATER+"
 		(shape passive)
 		(at 125.73 59.69 0)
-		(fields_autoplaced yes)
-		(effects
-			(font
-				(size 1.27 1.27)
-			)
-			(justify left)
-		)
-	)
-	(hierarchical_label "B2- (R)"
-		(shape passive)
-		(at 139.7 57.15 0)
 		(fields_autoplaced yes)
 		(effects
@@
 		)
 	)
-	(hierarchical_label "B2- (L)"
+	(hierarchical_label "B2-"
 		(shape passive)
 		(at 125.73 57.15 0)
@@
 		)
 	)
-	(hierarchical_label "B+ (L)"
+	(hierarchical_label "B+"
 		(shape passive)
 		(at 125.73 52.07 0)
@@
 		)
 	)
-	(hierarchical_label "HEATER- (L)"
+	(hierarchical_label "HEATER-"
 		(shape passive)
 		(at 125.73 62.23 0)
@@
 		)
 	)
-	(hierarchical_label "HEATER+ (R)"
-		(shape passive)
-		(at 142.24 59.69 0)
-		(fields_autoplaced yes)
-		(effects
-			(font
-				(size 1.27 1.27)
-			)
-			(justify left)
-		)
-	)
-	(hierarchical_label "B- (R)"
-		(shape passive)
-		(at 139.7 54.61 0)
-		(fields_autoplaced yes)
-		(effects
-			(font
-				(size 1.27 1.27)
-			)
-			(justify left)
-		)
-	)
-	(hierarchical_label "B+ (R)"
-		(shape passive)
-		(at 139.7 52.07 0)
-		(fields_autoplaced yes)
-		(effects
-			(font
-				(size 1.27 1.27)
-			)
-			(justify left)
-		)
-	)
-	(hierarchical_label "B- (L)"
+	(hierarchical_label "B-"
 		(shape passive)
 		(at 125.73 54.61 0)

Commit message: up
Changed lines of the file:
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@@
 		)
 	)
-	(hierarchical_label "HEATER-"
+	(hierarchical_label "GND{slash}HEATER-"
 		(shape passive)
 		(at 125.73 62.23 0)
